File: ebaz4205/components/ACOI.kicad_sch (KiCad schematic)
At the start: 1 part

Commit message: Consolidated all custom symbols into single library.
Library is available at ebaz4205/components/ebaz4205.kicad_sym

The templates and the schematics have been updated to use this library.
Keeping the original libraries for future reference.
Parts:
- removed U?: TPS3839DBZ, Package_TO_SOT_SMD:SOT-23, symbol Power_Supervisor:TPS3839DBZ
- added U?: TPS3839DBZ, Package_TO_SOT_SMD:SOT-23, symbol ebaz4205:TPS3839DBZ
Connections:
- net 1: now also U?.1 (GND)
- net 2: now also U?.2 (~RESET)
- net 3: now also U?.3 (VDD)
Changed lines of the file:
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@@
     (effects (font (size 1.27 1.27)) (justify left))
   )
-  (symbol (lib_id "Power_Supervisor:TPS3839DBZ") (at 12.7 20.32 0) (unit 1)
+  (symbol (lib_id "ebaz4205:TPS3839DBZ") (at 12.7 20.32 0) (unit 1)
     (in_bom yes) (on_board yes)
     (property "Reference" "U?" (id 0) (at 15.24 11.43 0)
@@
   )
   (symbol_instances
-    (path "/ee772e5f-26ec-4fab-9f50-54cbb8b805a5"
+    (path "/b21b14e0-a753-447e-a27f-00ad1219b43f"
       (reference "U?") (unit 1) (value "TPS3839DBZ") (footprint "Package_TO_SOT_SMD:SOT-23")
     )
