File: ebaz4205/components/L6.kicad_sch (KiCad schematic)
At the start: 1 part

Commit message: Consolidated all custom symbols into single library.
Library is available at ebaz4205/components/ebaz4205.kicad_sym

The templates and the schematics have been updated to use this library.
Keeping the original libraries for future reference.
Parts:
- removed LED?: LED_dual, symbol led:LED_dual
- added LED?: LED_dual, symbol ebaz4205:LED_dual
Connections:
- net 1: now also LED?.1 (A1)
- net 2: now also LED?.2 (A2)
- net 3: now also LED?.3 (K2)
- net 4: now also LED?.4 (K1)
Changed lines of the file:
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@@
     (effects (font (size 1.27 1.27)) (justify left))
   )
-  (symbol (lib_id "led:LED_dual") (at 19.05 12.7 0) (unit 1)
+  (symbol (lib_id "ebaz4205:LED_dual") (at 19.05 12.7 0) (unit 1)
     (in_bom yes) (on_board yes)
     (property "Reference" "LED?" (id 0) (at 19.05 1.27 0))
@@
   )
   (symbol_instances
-    (path "/4f07d0b9-6382-4f67-aa08-10252bfbe8a1"
+    (path "/a0b86502-3d7d-4dda-b6f5-e651bf2595fd"
       (reference "LED?") (unit 1) (value "LED_dual") (footprint "")
     )
