File: ebaz4205/components/U23.kicad_sch (KiCad schematic)
At the start: 1 part

Commit message: Consolidated all custom symbols into single library.
Library is available at ebaz4205/components/ebaz4205.kicad_sym

The templates and the schematics have been updated to use this library.
Keeping the original libraries for future reference.
Parts:
- removed U?: U23, symbol unknown:U23
- added U?: U23, symbol ebaz4205:U23
Connections:
- net 1: now also U?.1
- net 2: now also U?.2
- net 3: now also U?.3
- net 4: now also U?.4
Changed lines of the file:
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@@
     (effects (font (size 1.27 1.27)) (justify left))
   )
-  (symbol (lib_id "unknown:U23") (at 20.32 11.43 0) (unit 1)
+  (symbol (lib_id "ebaz4205:U23") (at 20.32 11.43 0) (unit 1)
     (in_bom yes) (on_board yes)
     (property "Reference" "U?" (id 0) (at 15.24 5.08 0)
@@
   )
   (symbol_instances
-    (path "/819a95ff-7c90-46bd-b8f0-45c29b4ca60e"
+    (path "/5571fc52-9b6f-48b2-8ed9-c8a5777816ff"
       (reference "U?") (unit 1) (value "U23") (footprint "")
     )
