File: ebaz4205/components/W29N01HVSINA.kicad_sch (KiCad schematic)
At the start: 1 part

Commit message: Consolidated all custom symbols into single library.
Library is available at ebaz4205/components/ebaz4205.kicad_sym

The templates and the schematics have been updated to use this library.
Keeping the original libraries for future reference.
Parts:
- removed IC?: W29N01HVSINA, SOP50P2000X120-48N, symbol W29N01HVSINA:W29N01HVSINA
- added IC?: W29N01HVSINA, SOP50P2000X120-48N, symbol ebaz4205:W29N01HVSINA
Connections:
- net 1: now also IC?.1 (N.C_1)
- net 10: now also IC?.10 (N.C_7)
- net 11: now also IC?.11 (N.C_8)
- net 12: now also IC?.12 (VCC_1)
- net 13: now also IC?.13 (VSS_1)
- net 14: now also IC?.14 (N.C_9)
- net 15: now also IC?.15 (N.C_10)
- net 16: now also IC?.16 (CLE)
- net 17: now also IC?.17 (ALE)
- net 18: now also IC?.18 (#WE)
- net 19: now also IC?.19 (#WP)
- net 2: now also IC?.2 (N.C_2)
- net 20: now also IC?.20 (DNU_1)
- net 21: now also IC?.21 (N.C_11)
- net 22: now also IC?.22 (N.C_12)
- net 23: now also IC?.23 (N.C_13)
- net 24: now also IC?.24 (N.C_14)
- net 25: now also IC?.25 (N.C_15)
- net 26: now also IC?.26 (N.C_16)
- net 27: now also IC?.27 (N.C_17)
- net 28: now also IC?.28 (N.C_18)
- net 29: now also IC?.29 (IO0)
- net 3: now also IC?.3 (N.C_3)
- net 30: now also IC?.30 (IO1)
- net 31: now also IC?.31 (IO2)
- net 32: now also IC?.32 (IO3)
- net 33: now also IC?.33 (N.C_19)
- net 34: now also IC?.34 (N.C_20)
- net 35: now also IC?.35 (N.C_21)
- net 36: now also IC?.36 (VSS_2)
- net 37: now also IC?.37 (VCC_2)
- net 38: now also IC?.38 (DNU_2)
- net 39: now also IC?.39 (N.C_22)
- net 4: now also IC?.4 (N.C_4)
- net 40: now also IC?.40 (N.C_23)
- net 41: now also IC?.41 (IO4)
- net 42: now also IC?.42 (IO5)
- net 43: now also IC?.43 (IO6)
- net 44: now also IC?.44 (IO7)
- net 45: now also IC?.45 (N.C_24)
- net 46: now also IC?.46 (N.C_25)
- net 47: now also IC?.47 (N.C_26)
- net 48: now also IC?.48 (N.C_27)
- net 5: now also IC?.5 (N.C_5)
- net 6: now also IC?.6 (N.C_6)
- net 7: now also IC?.7 (RY/#BY)
- net 8: now also IC?.8 (#RE)
- net 9: now also IC?.9 (#CE)
Changed lines of the file:
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@@
     (effects (font (size 1.27 1.27)) (justify left))
   )
-  (symbol (lib_id "W29N01HVSINA:W29N01HVSINA") (at 20.32 10.16 0) (unit 1)
+  (symbol (lib_id "ebaz4205:W29N01HVSINA") (at 20.32 10.16 0) (unit 1)
     (in_bom yes) (on_board yes)
     (property "Reference" "IC?" (id 0) (at 49.53 2.54 0)
@@
   )
   (symbol_instances
-    (path "/f8dc103b-9f13-4a45-92f7-e5f24ef0cf75"
+    (path "/0e5e40cb-92aa-42c9-981e-459ad0104c48"
       (reference "IC?") (unit 1) (value "W29N01HVSINA") (footprint "SOP50P2000X120-48N")
     )
