File: ebaz4205/components/dcdc.kicad_sch (KiCad schematic)
At the start: 1 part

Commit message: Consolidated all custom symbols into single library.
Library is available at ebaz4205/components/ebaz4205.kicad_sym

The templates and the schematics have been updated to use this library.
Keeping the original libraries for future reference.
Parts:
- removed U?: J37I, symbol dcdc:J37I
- added U?: J37I, symbol ebaz4205:J37I
Connections:
- net 1: now also U?.1 (GND)
- net 2: now also U?.2 (SW)
- net 3: now also U?.3 (IN)
- net 4: now also U?.4 (FB)
- net 5: now also U?.5 (EN)
- net 6: now also U?.6 (S)
Changed lines of the file:
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@@
     (effects (font (size 1.27 1.27)) (justify left))
   )
-  (symbol (lib_id "dcdc:J37I") (at 24.13 24.13 0) (unit 1)
+  (symbol (lib_id "ebaz4205:J37I") (at 24.13 24.13 0) (unit 1)
     (in_bom yes) (on_board yes)
     (property "Reference" "U?" (id 0) (at 16.51 13.97 0)
@@
   )
   (symbol_instances
-    (path "/f251107d-b8e0-40c9-acd6-a86385a2ebd1"
+    (path "/a6023c28-d335-409b-a393-868a17afea70"
       (reference "U?") (unit 1) (value "J37I") (footprint "")
     )
