File: ebaz4205/components/ddr_term.kicad_sch (KiCad schematic)
At the start: 1 part

Commit message: Consolidated all custom symbols into single library.
Library is available at ebaz4205/components/ebaz4205.kicad_sym

The templates and the schematics have been updated to use this library.
Keeping the original libraries for future reference.
Parts:
- removed IC?: TPS51200AQDRCRQ1, TPS51200AQDRCRQ1, symbol TPS51200AQDRCRQ1:TPS51200AQDRCRQ1
- added IC?: TPS51200AQDRCRQ1, TPS51200AQDRCRQ1, symbol ebaz4205:TPS51200AQDRCRQ1
Connections:
- net 1: now also IC?.1 (REFIN)
- net 10: now also IC?.10 (VIN)
- net 11: now also IC?.11 (EP_3)
- net 12: now also IC?.12 (EP_4)
- net 13: now also IC?.13 (EP_1)
- net 14: now also IC?.14 (EP_2)
- net 15: now also IC?.15 (EP_5)
- net 2: now also IC?.2 (VLDOIN)
- net 3: now also IC?.3 (VO)
- net 4: now also IC?.4 (PGND)
- net 5: now also IC?.5 (VOSNS)
- net 6: now also IC?.6 (REFOUT)
- net 7: now also IC?.7 (EN)
- net 8: now also IC?.8 (GND)
- net 9: now also IC?.9 (PGOOD)
Changed lines of the file:
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@@
     (effects (font (size 1.27 1.27)) (justify left))
   )
-  (symbol (lib_id "TPS51200AQDRCRQ1:TPS51200AQDRCRQ1") (at 34.29 31.75 0) (unit 1)
+  (symbol (lib_id "ebaz4205:TPS51200AQDRCRQ1") (at 34.29 31.75 0) (unit 1)
     (in_bom yes) (on_board yes)
     (property "Reference" "IC?" (id 0) (at 40.64 15.24 0)
@@
   )
   (symbol_instances
-    (path "/97fd596c-98c4-4e5f-92eb-2c7af2f5fec3"
+    (path "/1c629502-4b99-4081-97e9-b3b31de977db"
       (reference "IC?") (unit 1) (value "TPS51200AQDRCRQ1") (footprint "TPS51200AQDRCRQ1")
     )
