File: ebaz4205/components/dram.kicad_sch (KiCad schematic)
At the start: 2 parts

Commit message: Consolidated all custom symbols into single library.
Library is available at ebaz4205/components/ebaz4205.kicad_sym

The templates and the schematics have been updated to use this library.
Keeping the original libraries for future reference.
Parts:
- removed U? (x2): MT41K128M16JT-125_AITK, Micron-JT-0-0-*, symbol eec:MT41K128M16JT-125_AITK
- added U? (x2): MT41K128M16JT-125_AITK, Micron-JT-0-0-*, symbol ebaz4205:MT41K128M16JT-125_AITK
Connections:
- net A1: now also U?.A1 (VDDQ)
- net A2: now also U?.A2 (DQ13)
- net A3: now also U?.A3 (DQ15)
- net A7: now also U?.A7 (DQ12)
- net A8: now also U?.A8 (VDDQ)
- net A9: now also U?.A9 (VSS)
- net B1: now also U?.B1 (VSSQ)
- net B2: now also U?.B2 (VDD)
- net B3: now also U?.B3 (VSS)
- net B7: now also U?.B7 (~UDQS~)
- net B8: now also U?.B8 (DQ14)
- net B9: now also U?.B9 (VSSQ)
- net C1: now also U?.C1 (VDDQ)
- net C2: now also U?.C2 (DQ11)
- net C3: now also U?.C3 (DQ9)
- net C7: now also U?.C7 (UDQS)
- net C8: now also U?.C8 (DQ10)
- net C9: now also U?.C9 (VDDQ)
- net D1: now also U?.D1 (VSSQ)
- net D2: now also U?.D2 (VDDQ)
- net D3: now also U?.D3 (UDM)
- net D7: now also U?.D7 (DQ8)
- net D8: now also U?.D8 (VSSQ)
- net D9: now also U?.D9 (VDD)
- net E1: now also U?.E1 (VSS)
- net E2: now also U?.E2 (VSSQ)
- net E3: now also U?.E3 (DQ0)
- net E7: now also U?.E7 (LDM)
- net E8: now also U?.E8 (VSSQ)
- net E9: now also U?.E9 (VDDQ)
- net F1: now also U?.F1 (VDDQ)
- net F2: now also U?.F2 (DQ2)
- net F3: now also U?.F3 (LDQS)
- net F7: now also U?.F7 (DQ1)
- net F8: now also U?.F8 (DQ3)
- net F9: now also U?.F9 (VSSQ)
- net G1: now also U?.G1 (VSSQ)
- net G2: now also U?.G2 (DQ6)
- net G3: now also U?.G3 (~LDQS~)
- net G7: now also U?.G7 (VDD)
- net G8: now also U?.G8 (VSS)
- net G9: now also U?.G9 (VSSQ)
- net H1: now also U?.H1 (VREFDQ)
- net H2: now also U?.H2 (VDDQ)
- net H3: now also U?.H3 (DQ4)
- net H7: now also U?.H7 (DQ7)
- net H8: now also U?.H8 (DQ5)
- net H9: now also U?.H9 (VDDQ)
- net J1: now also U?.J1 (NC)
- net J2: now also U?.J2 (VSS)
- net J3: now also U?.J3 (~RAS~)
- net J7: now also U?.J7 (CK)
- net J8: now also U?.J8 (VSS)
- net J9: now also U?.J9 (NC)
- net K1: now also U?.K1 (ODT)
- net K2: now also U?.K2 (VDD)
- net K3: now also U?.K3 (~CAS~)
- net K7: now also U?.K7 (~CK~)
- net K8: now also U?.K8 (VDD)
- net K9: now also U?.K9 (CKE)
- net L1: now also U?.L1 (NC)
- net L2: now also U?.L2 (~CS~)
- net L3: now also U?.L3 (~WE~)
- net L7: now also U?.L7 (A10/AP)
- net L8: now also U?.L8 (ZQ)
- net L9: now also U?.L9 (NC)
- net M1: now also U?.M1 (VSS)
- net M2: now also U?.M2 (BA0)
- net M3: now also U?.M3 (BA2)
- net M7: now also U?.M7 (NC)
- net M8: now also U?.M8 (VREFCA)
- net M9: now also U?.M9 (VSS)
- net N1: now also U?.N1 (VDD)
- net N2: now also U?.N2 (A3)
- net N3: now also U?.N3 (A0)
- net N7: now also U?.N7 (A12/~BC~)
- net N8: now also U?.N8 (BA1)
- net N9: now also U?.N9 (VDD)
- net P1: now also U?.P1 (VSS)
- net P2: now also U?.P2 (A5)
- net P3: now also U?.P3 (A2)
- net P7: now also U?.P7 (A1)
- net P8: now also U?.P8 (A4)
- net P9: now also U?.P9 (VSS)
- net R1: now also U?.R1 (VDD)
- net R2: now also U?.R2 (A7)
- net R3: now also U?.R3 (A9)
- net R7: now also U?.R7 (A11)
- net R8: now also U?.R8 (A6)
- net R9: now also U?.R9 (VDD)
- net T1: now also U?.T1 (VSS)
- net T2: now also U?.T2 (~RESET~)
- net T3: now also U?.T3 (A13)
- net T7: now also U?.T7 (NC)
- net T8: now also U?.T8 (A8)
- net T9: now also U?.T9 (VSS)
Changed lines of the file:
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@@
     (effects (font (size 1.27 1.27)) (justify left))
   )
-  (symbol (lib_id "eec:MT41K128M16JT-125_AITK") (at 26.67 13.97 0) (unit 1)
+  (symbol (lib_id "ebaz4205:MT41K128M16JT-125_AITK") (at 26.67 13.97 0) (unit 1)
     (in_bom yes) (on_board yes)
     (property "Reference" "U?" (id 0) (at 26.67 8.89 0)
@@
     )
   )
-  (symbol (lib_id "eec:MT41K128M16JT-125_AITK") (at 85.09 13.97 0) (unit 2)
+  (symbol (lib_id "ebaz4205:MT41K128M16JT-125_AITK") (at 85.09 13.97 0) (unit 2)
     (in_bom yes) (on_board yes)
     (property "Reference" "U?" (id 0) (at 85.09 8.89 0)
@@
   )
   (symbol_instances
-    (path "/2c2f22ef-341a-4075-bac5-622a8d9fa374"
+    (path "/b98b90ab-a4f5-41a5-825a-68ac08ea761c"
       (reference "U?") (unit 1) (value "MT41K128M16JT-125_AITK") (footprint "Micron-JT-0-0-*")
     )
-    (path "/d9831f70-dc82-4019-9086-9eefaa4879a8"
+    (path "/23732892-e64c-4f14-96b6-7af39ceb6332"
       (reference "U?") (unit 2) (value "MT41K128M16JT-125_AITK") (footprint "Micron-JT-0-0-*")
     )
