File: ebaz4205/components/eth_transformer.kicad_sch (KiCad schematic)
At the start: 1 part

Commit message: Consolidated all custom symbols into single library.
Library is available at ebaz4205/components/ebaz4205.kicad_sym

The templates and the schematics have been updated to use this library.
Keeping the original libraries for future reference.
Parts:
- removed T?: HST-0041SAR, symbol trafo:HST-0041SAR
- added T?: HST-0041SAR, symbol ebaz4205:HST-0041SAR
Connections:
- net 1: now also T?.1 (TD+)
- net 10: now also T?.10 (RXCT)
- net 11: now also T?.11 (RX+)
- net 14: now also T?.14 (TX-)
- net 15: now also T?.15 (TXCT)
- net 16: now also T?.16 (TX+)
- net 2: now also T?.2 (TCT)
- net 3: now also T?.3 (TD-)
- net 6: now also T?.6 (RD+)
- net 7: now also T?.7 (RCT)
- net 8: now also T?.8 (RD-)
- net 9: now also T?.9 (RX-)
Changed lines of the file:
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@@
     (effects (font (size 1.27 1.27)) (justify left))
   )
-  (symbol (lib_id "trafo:HST-0041SAR") (at 30.48 22.86 0) (unit 1)
+  (symbol (lib_id "ebaz4205:HST-0041SAR") (at 30.48 22.86 0) (unit 1)
     (in_bom yes) (on_board yes)
     (property "Reference" "T?" (id 0) (at 30.48 3.175 0))
@@
   )
   (symbol_instances
-    (path "/e48ad1d8-9262-4b7c-b25a-d9f8f2d330e4"
+    (path "/8fcc7767-69b2-40d1-bda5-4485b4e70619"
       (reference "T?") (unit 1) (value "HST-0041SAR") (footprint "")
     )
