File: ebaz4205/components/osc.kicad_sch (KiCad schematic)
At the start: 1 part

Commit message: Consolidated all custom symbols into single library.
Library is available at ebaz4205/components/ebaz4205.kicad_sym

The templates and the schematics have been updated to use this library.
Keeping the original libraries for future reference.
Parts:
- removed X?: TXC-7C, Oscillator:Oscillator_SMD_TXC_7C-4Pin_5.0x3.2mm, symbol Oscillator:TXC-7C
- added X?: TXC-7C, Oscillator:Oscillator_SMD_TXC_7C-4Pin_5.0x3.2mm, symbol ebaz4205:TXC-7C
Connections:
- net 1: now also X?.1 (EN)
- net 2: now also X?.2 (GND)
- net 3: now also X?.3 (OUT)
- net 4: now also X?.4 (Vdd)
Changed lines of the file:
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@@
     (effects (font (size 1.27 1.27)) (justify left))
   )
-  (symbol (lib_id "Oscillator:TXC-7C") (at 21.59 19.05 0) (unit 1)
+  (symbol (lib_id "ebaz4205:TXC-7C") (at 21.59 19.05 0) (unit 1)
     (in_bom yes) (on_board yes)
     (property "Reference" "X?" (id 0) (at 16.51 12.7 0)
@@
   )
   (symbol_instances
-    (path "/b298c0e7-919b-418b-b5b5-c0928fc08168"
+    (path "/f0419c64-88e1-4fdd-b97e-2216ef49ef9a"
       (reference "X?") (unit 1) (value "TXC-7C") (footprint "Oscillator:Oscillator_SMD_TXC_7C-4Pin_5.0x3.2mm")
     )
