File: ebaz4205/components/osc2.kicad_sch (KiCad schematic)
At the start: 1 part

Commit message: Consolidated all custom symbols into single library.
Library is available at ebaz4205/components/ebaz4205.kicad_sym

The templates and the schematics have been updated to use this library.
Keeping the original libraries for future reference.
Parts:
- removed X?: TXC-EBAZ, symbol osc:TXC-EBAZ
- added X?: TXC-EBAZ, symbol ebaz4205:TXC-EBAZ
Connections:
- net 1: now also X?.1 (EN)
- net 2: now also X?.2 (Vdd)
- net 3: now also X?.3 (OUT)
- net 4: now also X?.4 (GND)
Changed lines of the file:
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@@
     (effects (font (size 1.27 1.27)) (justify left))
   )
-  (symbol (lib_id "osc:TXC-EBAZ") (at 21.59 19.05 0) (unit 1)
+  (symbol (lib_id "ebaz4205:TXC-EBAZ") (at 21.59 19.05 0) (unit 1)
     (in_bom yes) (on_board yes)
     (property "Reference" "X?" (id 0) (at 17.78 12.7 0))
@@
   )
   (symbol_instances
-    (path "/ae63eb83-1e27-44f0-8dbd-87ddcce5d5a0"
+    (path "/03d4f010-fe8c-4b6e-a333-04227f2ab605"
       (reference "X?") (unit 1) (value "TXC-EBAZ") (footprint "")
     )
