File: ebaz4205/components/rtc.kicad_sch (KiCad schematic)
At the start: 1 part

Commit message: Consolidated all custom symbols into single library.
Library is available at ebaz4205/components/ebaz4205.kicad_sym

The templates and the schematics have been updated to use this library.
Keeping the original libraries for future reference.
Parts:
- removed IC?: DS1307Z+, SOIC127P600X175-8N, symbol DS1307Z+:DS1307Z+
- added IC?: DS1307Z+, SOIC127P600X175-8N, symbol ebaz4205:DS1307Z+
Connections:
- net 1: now also IC?.1 (X1)
- net 2: now also IC?.2 (X2)
- net 3: now also IC?.3 (VBAT)
- net 4: now also IC?.4 (GND)
- net 5: now also IC?.5 (SDA)
- net 6: now also IC?.6 (SCL)
- net 7: now also IC?.7 (SQW/OUT)
- net 8: now also IC?.8 (VCC)
Changed lines of the file:
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@@
     (effects (font (size 1.27 1.27)) (justify left))
   )
-  (symbol (lib_id "DS1307Z+:DS1307Z+") (at 17.78 11.43 0) (unit 1)
+  (symbol (lib_id "ebaz4205:DS1307Z+") (at 17.78 11.43 0) (unit 1)
     (in_bom yes) (on_board yes)
     (property "Reference" "IC?" (id 0) (at 46.99 3.81 0)
@@
   )
   (symbol_instances
-    (path "/1a2fe25b-95a4-457a-a3c1-14c40e796eea"
+    (path "/6b4337e8-de15-4572-a255-b1b9a091293f"
       (reference "IC?") (unit 1) (value "DS1307Z+") (footprint "SOIC127P600X175-8N")
     )
