File: ebaz4205/components/rtc_osc.kicad_sch (KiCad schematic)
At the start: 1 part

Commit message: Consolidated all custom symbols into single library.
Library is available at ebaz4205/components/ebaz4205.kicad_sym

The templates and the schematics have been updated to use this library.
Keeping the original libraries for future reference.
Parts:
- removed Y?: RTC_XTAL, symbol osc:RTC_XTAL
- added Y?: RTC_XTAL, symbol ebaz4205:RTC_XTAL
Connections:
- net 1: now also Y?.1
- net 2: now also Y?.2
- net 3: now also Y?.3
- net 4: now also Y?.4
- net 5: now also Y?.5
- net 6: now also Y?.6
- net 7: now also Y?.7
- net 8: now also Y?.8
Changed lines of the file:
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@@
     (effects (font (size 1.27 1.27)) (justify left))
   )
-  (symbol (lib_id "osc:RTC_XTAL") (at 25.4 31.75 0) (unit 1)
+  (symbol (lib_id "ebaz4205:RTC_XTAL") (at 25.4 31.75 0) (unit 1)
     (in_bom yes) (on_board yes)
     (property "Reference" "Y?" (id 0) (at 25.4 7.62 0))
@@
   )
   (symbol_instances
-    (path "/dbf9dd4d-61b7-4301-9531-21965f4d9e29"
+    (path "/e07edf04-01b1-4a56-b31b-6b42e5ac4a77"
       (reference "Y?") (unit 1) (value "RTC_XTAL") (footprint "")
     )
