File: ebaz4205/components/sd_card.kicad_sch (KiCad schematic)
At the start: 1 part

Commit message: Consolidated all custom symbols into single library.
Library is available at ebaz4205/components/ebaz4205.kicad_sym

The templates and the schematics have been updated to use this library.
Keeping the original libraries for future reference.
Parts:
- removed U?: Micro_SD_Card_mount, symbol sd_card:Micro_SD_Card_mount
- added U?: Micro_SD_Card_mount, symbol ebaz4205:Micro_SD_Card_mount
Connections:
- net 1: now also U?.1 (DAT2)
- net 10: now also U?.10 (MNT1)
- net 11: now also U?.11 (MNT2)
- net 12: now also U?.12 (MNT3)
- net 13: now also U?.13 (MNT4)
- net 2: now also U?.2 (DAT3/CD)
- net 3: now also U?.3 (CMD)
- net 4: now also U?.4 (VDD)
- net 5: now also U?.5 (CLK)
- net 6: now also U?.6 (VSS)
- net 7: now also U?.7 (DAT0)
- net 8: now also U?.8 (DAT1)
- net 9: now also U?.9 (DETECT)
Changed lines of the file:
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@@
     (effects (font (size 1.27 1.27)) (justify right))
   )
-  (symbol (lib_id "sd_card:Micro_SD_Card_mount") (at 41.91 17.78 0) (unit 1)
+  (symbol (lib_id "ebaz4205:Micro_SD_Card_mount") (at 41.91 17.78 0) (unit 1)
     (in_bom yes) (on_board yes)
     (property "Reference" "U?" (id 0) (at 22.86 2.54 0)
@@
   )
   (symbol_instances
-    (path "/3ad41296-4eb4-4c52-87e1-8ca5f9cee63d"
+    (path "/4c19a587-49b3-4617-bbf5-4bf8f3aec7f7"
       (reference "U?") (unit 1) (value "Micro_SD_Card_mount") (footprint "")
     )
