File: ebaz4205/components/supervisor.kicad_sch (KiCad schematic)
At the start: 1 part

Commit message: Consolidated all custom symbols into single library.
Library is available at ebaz4205/components/ebaz4205.kicad_sym

The templates and the schematics have been updated to use this library.
Keeping the original libraries for future reference.
Parts:
- removed U?: SGM706, symbol supervisor:SGM706
- added U?: SGM706, symbol ebaz4205:SGM706
Connections:
- net 1: now also U?.1 (~MR)
- net 2: now also U?.2 (VCC)
- net 3: now also U?.3 (GND)
- net 4: now also U?.4 (PFI)
- net 5: now also U?.5 (~PFO)
- net 6: now also U?.6 (WDI)
- net 7: now also U?.7 (~RESET)
- net 8: now also U?.8 (~WDO)
Changed lines of the file:
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@@
     (effects (font (size 1.27 1.27)) (justify left))
   )
-  (symbol (lib_id "supervisor:SGM706") (at 24.13 11.43 0) (unit 1)
+  (symbol (lib_id "ebaz4205:SGM706") (at 24.13 11.43 0) (unit 1)
     (in_bom yes) (on_board yes)
     (property "Reference" "U?" (id 0) (at 24.13 2.54 0))
@@
   )
   (symbol_instances
-    (path "/73f714df-baf2-4e40-af96-3b127a404e3e"
+    (path "/20cca72f-ebeb-433b-aae5-e4f48cc1f745"
       (reference "U?") (unit 1) (value "SGM706") (footprint "")
     )
