File: ebaz4205/components/xc7z010.kicad_sch (KiCad schematic)
At the start: 9 parts

Commit message: Provided all component symbols.
Symbol libraries are available as subdirectories in ebaz4205/components/

U23 is still unknown, so a placeholder symbol was provided.
Parts:
- removed U? (x9): xc7z010clg400, symbol xilinx7:xc7z010clg400
- added U? (x9): xc7z010clg400, symbol xilinx7:xc7z010clg400
Connections:
- net A1: now also U?.A1 (PS_DDR_DM0_502)
- net A10: now also U?.A10 (PS_MIO37_501)
- net A11: now also U?.A11 (PS_MIO36_501)
- net A12: now also U?.A12 (PS_MIO34_501)
- net A13: now also U?.A13 (VCCO_MIO1_501[4]), U?.B16 (VCCO_MIO1_501[4]), U?.D12 (VCCO_MIO1_501[4]), U?.E15 (VCCO_MIO1_501[4])
- net A14: now also U?.A14 (PS_MIO32_501)
- net A15: now also U?.A15 (PS_MIO26_501)
- net A16: now also U?.A16 (PS_MIO24_501)
- net A17: now also U?.A17 (PS_MIO20_501)
- net A19: now also U?.A19 (PS_MIO16_501)
- net A2: now also U?.A2 (PS_DDR_DQ2_502)
- net A20: now also U?.A20 (IO_L2N_T0_AD8N_35)
- net A3: now also U?.A3 (VCCO_DDR_502[10]), U?.D2 (VCCO_DDR_502[10]), U?.E5 (VCCO_DDR_502[10]), U?.G1 (VCCO_DDR_502[10]), U?.H4 (VCCO_DDR_502[10]), U?.L3 (VCCO_DDR_502[10]), U?.P2 (VCCO_DDR_502[10]), U?.R5 (VCCO_DDR_502[10]), U?.U1 (VCCO_DDR_502[10]), U?.V4 (VCCO_DDR_502[10])
- net A4: now also U?.A4 (PS_DDR_DQ3_502)
- net A5: now also U?.A5 (PS_MIO6_500)
- net A6: now also U?.A6 (PS_MIO5_500)
- net A7: now also U?.A7 (PS_MIO1_500)
- net A8: now also U?.A18 (GND[59]), U?.A8 (GND[59]), U?.B1 (GND[59]), U?.B11 (GND[59]), U?.C14 (GND[59]), U?.C4 (GND[59]), U?.C9 (GND[59]), U?.D17 (GND[59]), U?.E10 (GND[59]), U?.E20 (GND[59]), U?.F3 (GND[59]), U?.F7 (GND[59]), U?.G10 (GND[59]), U?.G12 (GND[59]), U?.G16 (GND[59]), U?.H11 (GND[59]), U?.H13 (GND[59]), U?.H19 (GND[59]), U?.H7 (GND[59]), U?.H9 (GND[59]), U?.J12 (GND[59]), U?.J2 (GND[59]), U?.J8 (GND[59]), U?.K11 (GND[59]), U?.K13 (GND[59]), U?.K15 (GND[59]), U?.K5 (GND[59]), U?.K7 (GND[59]), U?.L12 (GND[59]), U?.L18 (GND[59]), U?.L8 (GND[59]), U?.M1 (GND[59]), U?.M11 (GND[59]), U?.M13 (GND[59]), U?.M7 (GND[59]), U?.N10 (GND[59]), U?.N12 (GND[59]), U?.N14 (GND[59]), U?.N4 (GND[59]), U?.N8 (GND[59]), U?.P11 (GND[59]), U?.P13 (GND[59]), U?.P17 (GND[59]), U?.P7 (GND[59]), U?.P9 (GND[59]), U?.R12 (GND[59]), U?.R20 (GND[59]), U?.R8 (GND[59]), U?.T13 (GND[59]), U?.T3 (GND[59]), U?.T7 (GND[59]), U?.U16 (GND[59]), U?.U6 (GND[59]), U?.V19 (GND[59]), U?.V9 (GND[59]), U?.W12 (GND[59]), U?.W2 (GND[59]), U?.Y15 (GND[59]), U?.Y5 (GND[59])
- net A9: now also U?.A9 (PS_MIO43_501)
- net B10: now also U?.B10 (PS_SRST_B_501)
- net B12: now also U?.B12 (PS_MIO48_501)
- net B13: now also U?.B13 (PS_MIO50_501)
- net B14: now also U?.B14 (PS_MIO47_501)
- net B15: now also U?.B15 (PS_MIO45_501)
- net B17: now also U?.B17 (PS_MIO22_501)
- net B18: now also U?.B18 (PS_MIO18_501)
- net B19: now also U?.B19 (IO_L2P_T0_AD8P_35)
- net B2: now also U?.B2 (PS_DDR_DQS_N0_502)
- net B20: now also U?.B20 (IO_L1N_T0_AD0N_35)
- net B3: now also U?.B3 (PS_DDR_DQ1_502)
- net B4: now also U?.B4 (PS_DDR_DRST_B_502)
- net B5: now also U?.B5 (PS_MIO9_500)
- net B6: now also U?.B6 (VCCO_MIO0_500[2]), U?.D7 (VCCO_MIO0_500[2])
- net B7: now also U?.B7 (PS_MIO4_500)
- net B8: now also U?.B8 (PS_MIO2_500)
- net B9: now also U?.B9 (PS_MIO51_501)
- net C1: now also U?.C1 (PS_DDR_DQ6_502)
- net C10: now also U?.C10 (PS_MIO52_501)
- net C11: now also U?.C11 (PS_MIO53_501)
- net C12: now also U?.C12 (PS_MIO49_501)
- net C13: now also U?.C13 (PS_MIO29_501)
- net C15: now also U?.C15 (PS_MIO30_501)
- net C16: now also U?.C16 (PS_MIO28_501)
- net C17: now also U?.C17 (PS_MIO41_501)
- net C18: now also U?.C18 (PS_MIO39_501)
- net C19: now also U?.C19 (VCCO_35[6]), U?.F18 (VCCO_35[6]), U?.H14 (VCCO_35[6]), U?.J17 (VCCO_35[6]), U?.K20 (VCCO_35[6]), U?.M16 (VCCO_35[6])
- net C2: now also U?.C2 (PS_DDR_DQS_P0_502)
- net C20: now also U?.C20 (IO_L1P_T0_AD0P_35)
- net C3: now also U?.C3 (PS_DDR_DQ0_502)
- net C5: now also U?.C5 (PS_MIO14_500)
- net C6: now also U?.C6 (PS_MIO11_500)
- net C7: now also U?.C7 (PS_POR_B_500)
- net C8: now also U?.C8 (PS_MIO15_500)
- net D1: now also U?.D1 (PS_DDR_DQ5_502)
- net D10: now also U?.D10 (PS_MIO19_501)
- net D11: now also U?.D11 (PS_MIO23_501)
- net D13: now also U?.D13 (PS_MIO27_501)
- net D14: now also U?.D14 (PS_MIO40_501)
- net D15: now also U?.D15 (PS_MIO33_501)
- net D16: now also U?.D16 (PS_MIO46_501)
- net D18: now also U?.D18 (IO_L3N_T0_DQS_AD1N_35)
- net D19: now also U?.D19 (IO_L4P_T0_35)
- net D20: now also U?.D20 (IO_L4N_T0_35)
- net D3: now also U?.D3 (PS_DDR_DQ4_502)
- net D4: now also U?.D4 (PS_DDR_A13_502)
- net D5: now also U?.D5 (PS_MIO8_500)
- net D6: now also U?.D6 (PS_MIO3_500)
- net D8: now also U?.D8 (PS_MIO7_500)
- net D9: now also U?.D9 (PS_MIO12_500)
- net E1: now also U?.E1 (PS_DDR_DQ7_502)
- net E11: now also U?.E11 (PS_MIO_VREF_501)
- net E12: now also U?.E12 (PS_MIO42_501)
- net E13: now also U?.E13 (PS_MIO38_501)
- net E14: now also U?.E14 (PS_MIO17_501)
- net E16: now also U?.E16 (PS_MIO31_501)
- net E17: now also U?.E17 (IO_L3P_T0_DQS_AD1P_35)
- net E18: now also U?.E18 (IO_L5P_T0_AD9P_35)
- net E19: now also U?.E19 (IO_L5N_T0_AD9N_35)
- net E2: now also U?.E2 (PS_DDR_DQ8_502)
- net E3: now also U?.E3 (PS_DDR_DQ9_502)
- net E4: now also U?.E4 (PS_DDR_A12_502)
- net E6: now also U?.E6 (PS_MIO0_500)
- net E7: now also U?.E7 (PS_CLK_500)
- net E8: now also U?.E8 (PS_MIO13_500)
- net E9: now also U?.E9 (PS_MIO10_500)
- net F1: now also U?.F1 (PS_DDR_DM1_502)
- net F10: now also U?.F10 (RSVDGND)
- net F11: now also U?.F11 (VCCBATT_0)
- net F12: now also U?.F12 (PS_MIO35_501)
- net F13: now also U?.F13 (PS_MIO44_501)
- net F14: now also U?.F14 (PS_MIO21_501)
- net F15: now also U?.F15 (PS_MIO25_501)
- net F16: now also U?.F16 (IO_L6P_T0_35)
- net F17: now also U?.F17 (IO_L6N_T0_VREF_35)
- net F19: now also U?.F19 (IO_L15P_T2_DQS_AD12P_35)
- net F2: now also U?.F2 (PS_DDR_DQS_N1_502)
- net F20: now also U?.F20 (IO_L15N_T2_DQS_AD12N_35)
- net F4: now also U?.F4 (PS_DDR_A14_502)
- net F5: now also U?.F5 (PS_DDR_A10_502)
- net F6: now also U?.F6 (TDO_0)
- net F9: now also U?.F9 (TCK_0)
- net G11: now also U?.G11 (VCCBRAM[2]), U?.H10 (VCCBRAM[2])
- net G13: now also U?.G13 (VCCINT[9]), U?.H12 (VCCINT[9]), U?.J13 (VCCINT[9]), U?.K12 (VCCINT[9]), U?.L13 (VCCINT[9]), U?.M12 (VCCINT[9]), U?.N13 (VCCINT[9]), U?.P12 (VCCINT[9]), U?.R13 (VCCINT[9])
- net G14: now also U?.G14 (IO_0_35)
- net G15: now also U?.G15 (IO_L19N_T3_VREF_35)
- net G17: now also U?.G17 (IO_L16P_T2_35)
- net G18: now also U?.G18 (IO_L16N_T2_35)
- net G19: now also U?.G19 (IO_L18P_T2_AD13P_35)
- net G2: now also U?.G2 (PS_DDR_DQS_P1_502)
- net G20: now also U?.G20 (IO_L18N_T2_AD13N_35)
- net G3: now also U?.G3 (PS_DDR_DQ10_502)
- net G4: now also U?.G4 (PS_DDR_A11_502)
- net G5: now also U?.G5 (PS_DDR_VRN_502)
- net G6: now also U?.G6 (TDI_0)
- net G7: now also U?.G7 (VCCPINT[6]), U?.J7 (VCCPINT[6]), U?.L7 (VCCPINT[6]), U?.N7 (VCCPINT[6]), U?.P8 (VCCPINT[6]), U?.R7 (VCCPINT[6])
- net G8: now also U?.G8 (VCCPLL)
- net G9: now also U?.F8 (VCCPAUX[5]), U?.G9 (VCCPAUX[5]), U?.H8 (VCCPAUX[5]), U?.K8 (VCCPAUX[5]), U?.M8 (VCCPAUX[5])
- net H1: now also U?.H1 (PS_DDR_DQ14_502)
- net H15: now also U?.H15 (IO_L19P_T3_35)
- net H16: now also U?.H16 (IO_L13P_T2_MRCC_35)
- net H17: now also U?.H17 (IO_L13N_T2_MRCC_35)
- net H18: now also U?.H18 (IO_L14N_T2_AD4N_SRCC_35)
- net H2: now also U?.H2 (PS_DDR_DQ13_502)
- net H20: now also U?.H20 (IO_L17N_T2_AD5N_35)
- net H3: now also U?.H3 (PS_DDR_DQ11_502)
- net H5: now also U?.H5 (PS_DDR_VRP_502)
- net H6: now also U?.H6 (PS_DDR_VREF0_502)
- net J1: now also U?.J1 (PS_DDR_DQ15_502)
- net J10: now also U?.J10 (GNDADC_0)
- net J11: now also U?.J11 (VCCAUX[6]), U?.L11 (VCCAUX[6]), U?.N11 (VCCAUX[6]), U?.N9 (VCCAUX[6]), U?.P10 (VCCAUX[6]), U?.R9 (VCCAUX[6])
- net J14: now also U?.J14 (IO_L20N_T3_AD6N_35)
- net J15: now also U?.J15 (IO_25_35)
- net J16: now also U?.J16 (IO_L24N_T3_AD15N_35)
- net J18: now also U?.J18 (IO_L14P_T2_AD4P_SRCC_35)
- net J19: now also U?.J19 (IO_L10N_T1_AD11N_35)
- net J20: now also U?.J20 (IO_L17P_T2_AD5P_35)
- net J3: now also U?.J3 (PS_DDR_DQ12_502)
- net J4: now also U?.J4 (PS_DDR_A9_502)
- net J5: now also U?.J5 (PS_DDR_BA2_502)
- net J6: now also U?.J6 (TMS_0)
- net J9: now also U?.J9 (VCCADC_0)
- net K1: now also U?.K1 (PS_DDR_A8_502)
- net K10: now also U?.K10 (VREFN_0)
- net K14: now also U?.K14 (IO_L20P_T3_AD6P_35)
- net K16: now also U?.K16 (IO_L24P_T3_AD15P_35)
- net K17: now also U?.K17 (IO_L12P_T1_MRCC_35)
- net K18: now also U?.K18 (IO_L12N_T1_MRCC_35)
- net K19: now also U?.K19 (IO_L10P_T1_AD11P_35)
- net K2: now also U?.K2 (PS_DDR_A1_502)
- net K3: now also U?.K3 (PS_DDR_A3_502)
- net K4: now also U?.K4 (PS_DDR_A7_502)
- net K6: now also U?.K6 (VCCO_0)
- net K9: now also U?.K9 (VP_0)
- net L1: now also U?.L1 (PS_DDR_A5_502)
- net L10: now also U?.L10 (VN_0)
- net L14: now also U?.L14 (IO_L22P_T3_AD7P_35)
- net L15: now also U?.L15 (IO_L22N_T3_AD7N_35)
- net L16: now also U?.L16 (IO_L11P_T1_SRCC_35)
- net L17: now also U?.L17 (IO_L11N_T1_SRCC_35)
- net L19: now also U?.L19 (IO_L9P_T1_DQS_AD3P_35)
- net L2: now also U?.L2 (PS_DDR_CKP_502)
- net L20: now also U?.L20 (IO_L9N_T1_DQS_AD3N_35)
- net L4: now also U?.L4 (PS_DDR_A6_502)
- net L5: now also U?.L5 (PS_DDR_BA0_502)
- net L6: now also U?.L6 (PROGRAM_B_0)
- net L9: now also U?.L9 (VREFP_0)
- net M10: now also U?.M10 (DXN_0)
- net M14: now also U?.M14 (IO_L23P_T3_35)
- net M15: now also U?.M15 (IO_L23N_T3_35)
- net M17: now also U?.M17 (IO_L8P_T1_AD10P_35)
- net M18: now also U?.M18 (IO_L8N_T1_AD10N_35)
- net M19: now also U?.M19 (IO_L7P_T1_AD2P_35)
- net M2: now also U?.M2 (PS_DDR_CKN_502)
- net M20: now also U?.M20 (IO_L7N_T1_AD2N_35)
- net M3: now also U?.M3 (PS_DDR_A2_502)
- net M4: now also U?.M4 (PS_DDR_A4_502)
- net M5: now also U?.M5 (PS_DDR_WE_B_502)
- net M6: now also U?.M6 (CFGBVS_0)
- net M9: now also U?.M9 (DXP_0)
- net N1: now also U?.N1 (PS_DDR_CS_B_502)
- net N15: now also U?.N15 (IO_L21P_T3_DQS_AD14P_35)
- net N16: now also U?.N16 (IO_L21N_T3_DQS_AD14N_35)
- net N17: now also U?.N17 (IO_L23P_T3_34)
- net N18: now also U?.N18 (IO_L13P_T2_MRCC_34)
- net N19: now also U?.N19 (VCCO_34[6]), U?.R15 (VCCO_34[6]), U?.T18 (VCCO_34[6]), U?.V14 (VCCO_34[6]), U?.W17 (VCCO_34[6]), U?.Y20 (VCCO_34[6])
- net N2: now also U?.N2 (PS_DDR_A0_502)
- net N20: now also U?.N20 (IO_L14P_T2_SRCC_34)
- net N3: now also U?.N3 (PS_DDR_CKE_502)
- net N5: now also U?.N5 (PS_DDR_ODT_502)
- net N6: now also U?.N6 (RSVDVCC3)
- net P1: now also U?.P1 (PS_DDR_DQ16_502)
- net P14: now also U?.P14 (IO_L6P_T0_34)
- net P15: now also U?.P15 (IO_L24P_T3_34)
- net P16: now also U?.P16 (IO_L24N_T3_34)
- net P18: now also U?.P18 (IO_L23N_T3_34)
- net P19: now also U?.P19 (IO_L13N_T2_MRCC_34)
- net P20: now also U?.P20 (IO_L14N_T2_SRCC_34)
- net P3: now also U?.P3 (PS_DDR_DQ17_502)
- net P4: now also U?.P4 (PS_DDR_RAS_B_502)
- net P5: now also U?.P5 (PS_DDR_CAS_B_502)
- net P6: now also U?.P6 (PS_DDR_VREF1_502)
- net R1: now also U?.R1 (PS_DDR_DQ19_502)
- net R10: now also U?.R10 (INIT_B_0)
- net R11: now also U?.R11 (DONE_0)
- net R14: now also U?.R14 (IO_L6N_T0_VREF_34)
- net R16: now also U?.R16 (IO_L19P_T3_34)
- net R17: now also U?.R17 (IO_L19N_T3_VREF_34)
- net R18: now also U?.R18 (IO_L20N_T3_34)
- net R19: now also U?.R19 (IO_0_34)
- net R2: now also U?.R2 (PS_DDR_DQS_P2_502)
- net R3: now also U?.R3 (PS_DDR_DQ18_502)
- net R4: now also U?.R4 (PS_DDR_BA1_502)
- net R6: now also U?.R6 (RSVDVCC2)
- net T1: now also U?.T1 (PS_DDR_DM2_502)
- net T10: now also U?.T10 (IO_L1N_T0_34)
- net T11: now also U?.T11 (IO_L1P_T0_34)
- net T12: now also U?.T12 (IO_L2P_T0_34)
- net T14: now also U?.T14 (IO_L5P_T0_34)
- net T15: now also U?.T15 (IO_L5N_T0_34)
- net T16: now also U?.T16 (IO_L9P_T1_DQS_34)
- net T17: now also U?.T17 (IO_L20P_T3_34)
- net T19: now also U?.T19 (IO_25_34)
- net T2: now also U?.T2 (PS_DDR_DQS_N2_502)
- net T20: now also U?.T20 (IO_L15P_T2_DQS_34)
- net T4: now also U?.T4 (PS_DDR_DQ20_502)
- net T6: now also U?.T6 (RSVDVCC1)
- net T8: now also U?.T8 (VCCO_13[4]), U?.U11 (VCCO_13[4]), U?.W7 (VCCO_13[4]), U?.Y10 (VCCO_13[4])
- net U12: now also U?.U12 (IO_L2N_T0_34)
- net U13: now also U?.U13 (IO_L3P_T0_DQS_PUDC_B_34)
- net U14: now also U?.U14 (IO_L11P_T1_SRCC_34)
- net U15: now also U?.U15 (IO_L11N_T1_SRCC_34)
- net U17: now also U?.U17 (IO_L9N_T1_DQS_34)
- net U18: now also U?.U18 (IO_L12P_T1_MRCC_34)
- net U19: now also U?.U19 (IO_L12N_T1_MRCC_34)
- net U2: now also U?.U2 (PS_DDR_DQ22_502)
- net U20: now also U?.U20 (IO_L15N_T2_DQS_34)
- net U3: now also U?.U3 (PS_DDR_DQ23_502)
- net U4: now also U?.U4 (PS_DDR_DQ21_502)
- net V1: now also U?.V1 (PS_DDR_DQ24_502)
- net V12: now also U?.V12 (IO_L4P_T0_34)
- net V13: now also U?.V13 (IO_L3N_T0_DQS_34)
- net V15: now also U?.V15 (IO_L10P_T1_34)
- net V16: now also U?.V16 (IO_L18P_T2_34)
- net V17: now also U?.V17 (IO_L21P_T3_DQS_34)
- net V18: now also U?.V18 (IO_L21N_T3_DQS_34)
- net V2: now also U?.V2 (PS_DDR_DQ30_502)
- net V20: now also U?.V20 (IO_L16P_T2_34)
- net V3: now also U?.V3 (PS_DDR_DQ31_502)
- net W1: now also U?.W1 (PS_DDR_DQ26_502)
- net W13: now also U?.W13 (IO_L4N_T0_34)
- net W14: now also U?.W14 (IO_L8P_T1_34)
- net W15: now also U?.W15 (IO_L10N_T1_34)
- net W16: now also U?.W16 (IO_L18N_T2_34)
- net W18: now also U?.W18 (IO_L22P_T3_34)
- net W19: now also U?.W19 (IO_L22N_T3_34)
- net W20: now also U?.W20 (IO_L16N_T2_34)
- net W3: now also U?.W3 (PS_DDR_DQ29_502)
- net W4: now also U?.W4 (PS_DDR_DQS_N3_502)
- net W5: now also U?.W5 (PS_DDR_DQS_P3_502)
- net Y1: now also U?.Y1 (PS_DDR_DM3_502)
- net Y14: now also U?.Y14 (IO_L8N_T1_34)
- net Y16: now also U?.Y16 (IO_L7P_T1_34)
- net Y17: now also U?.Y17 (IO_L7N_T1_34)
- net Y18: now also U?.Y18 (IO_L17P_T2_34)
- net Y19: now also U?.Y19 (IO_L17N_T2_34)
- net Y2: now also U?.Y2 (PS_DDR_DQ28_502)
- net Y3: now also U?.Y3 (PS_DDR_DQ25_502)
- net Y4: now also U?.Y4 (PS_DDR_DQ27_502)
Changed lines of the file:
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@@
     )
   )
-  (symbol (lib_id "xilinx7:xc7z010clg400") (at 422.91 8.89 0) (unit 9)
+  (symbol (lib_id "xilinx7:xc7z010clg400") (at 425.45 8.89 0) (unit 9)
     (in_bom yes) (on_board yes)
-    (property "Reference" "U?" (id 0) (at 427.99 2.54 0)
+    (property "Reference" "U?" (id 0) (at 430.53 2.54 0)
       (effects (font (size 1.524 1.524)) (justify left))
     )
-    (property "Value" "xc7z010clg400" (id 1) (at 427.99 5.08 0)
+    (property "Value" "xc7z010clg400" (id 1) (at 430.53 5.08 0)
       (effects (font (size 1.524 1.524)) (justify left))
     )
-    (property "Footprint" "" (id 2) (at 427.99 7.62 0)
+    (property "Footprint" "" (id 2) (at 430.53 7.62 0)
       (effects (font (size 1.524 1.524)) (justify left) hide)
     )
-    (property "Datasheet" "" (id 3) (at 427.99 12.7 0)
+    (property "Datasheet" "" (id 3) (at 430.53 12.7 0)
       (effects (font (size 1.524 1.524)) (justify left) hide)
     )
-    (property "desc" "xc7z010clg400" (id 4) (at 427.99 15.24 0)
+    (property "desc" "xc7z010clg400" (id 4) (at 430.53 15.24 0)
       (effects (font (size 1.524 1.524)) (justify left) hide)
     )
@@
   )
   (symbol_instances
-    (path "/75ce1c41-58e5-4ce9-8d09-342d21d3ab2c"
+    (path "/1397eacc-3db6-4ed4-8a62-0dfb22424df0"
       (reference "U?") (unit 1) (value "xc7z010clg400") (footprint "")
     )
-    (path "/7fabca9c-7d52-417a-978c-9de0968580b4"
+    (path "/82397224-5b5c-49ec-a93b-0ae310f66c94"
       (reference "U?") (unit 2) (value "xc7z010clg400") (footprint "")
     )
-    (path "/f63a9cfd-f0a2-43e5-8363-55c3ff3fc252"
+    (path "/8a2f2c4e-0713-4cdb-826d-b28030feed98"
       (reference "U?") (unit 3) (value "xc7z010clg400") (footprint "")
     )
-    (path "/0aaf68bf-e290-4ebd-935d-005d0c171fb6"
+    (path "/556fb7d0-b037-4b5f-8b1b-b7f169fd683a"
       (reference "U?") (unit 4) (value "xc7z010clg400") (footprint "")
     )
-    (path "/4e1f6806-4db2-4e84-8ab7-aff3b55ea1ea"
+    (path "/6c0ff9ab-5622-4dce-88c2-4ff126cc5a3f"
       (reference "U?") (unit 5) (value "xc7z010clg400") (footprint "")
     )
-    (path "/46eaf245-652a-4a0c-b4c7-5691581572d8"
+    (path "/8f980645-5750-46fc-9dc7-6ed3528176cb"
       (reference "U?") (unit 6) (value "xc7z010clg400") (footprint "")
     )
-    (path "/10997501-e528-4d99-b860-869fb33a9e11"
+    (path "/76732ae3-5d45-4fb0-ba9c-5e2d9a365a79"
       (reference "U?") (unit 7) (value "xc7z010clg400") (footprint "")
     )
-    (path "/1141be2b-98b0-4bdc-bc4f-88745b920834"
+    (path "/5c78c30e-bf31-4039-ac4a-5d9b5e1e6aa4"
       (reference "U?") (unit 8) (value "xc7z010clg400") (footprint "")
     )
-    (path "/d96bc03f-ed27-451b-9816-e768144feaa7"
+    (path "/be912085-bcd1-40c7-91f9-0a007e125679"
       (reference "U?") (unit 9) (value "xc7z010clg400") (footprint "")
     )

Commit message: Added netlist - SchComponent pin checking. Fixed symbols.
Rebuilt Xilinx symbol without bundling.
Parts:
- removed U? (x9): xc7z010clg400, symbol xilinx7:xc7z010clg400
- added U? (x9): xc7z010clg400, symbol xilinx7:xc7z010clg400
Connections:
- net A1: now also U?.A1 (PS_DDR_DM0_502)
- net A10: now also U?.A10 (PS_MIO37_501)
- net A11: now also U?.A11 (PS_MIO36_501)
- net A12: now also U?.A12 (PS_MIO34_501)
- net A13: now also U?.A13 (VCCO_MIO1_501)
- net A14: now also U?.A14 (PS_MIO32_501)
- net A15: now also U?.A15 (PS_MIO26_501)
- net A16: now also U?.A16 (PS_MIO24_501)
- net A17: now also U?.A17 (PS_MIO20_501)
- net A19: now also U?.A19 (PS_MIO16_501)
- net A2: now also U?.A2 (PS_DDR_DQ2_502)
- net A20: now also U?.A20 (IO_L2N_T0_AD8N_35)
- net A3: now also U?.A3 (VCCO_DDR_502)
- net A4: now also U?.A4 (PS_DDR_DQ3_502)
- net A5: now also U?.A5 (PS_MIO6_500)
- net A6: now also U?.A6 (PS_MIO5_500)
- net A7: now also U?.A7 (PS_MIO1_500)
- net A8: now also U?.A8 (GND)
- net A9: now also U?.A9 (PS_MIO43_501)
- net B10: now also U?.B10 (PS_SRST_B_501)
- net B12: now also U?.B12 (PS_MIO48_501)
- net B13: now also U?.B13 (PS_MIO50_501)
- net B14: now also U?.B14 (PS_MIO47_501)
- net B15: now also U?.B15 (PS_MIO45_501)
- net B17: now also U?.B17 (PS_MIO22_501)
- net B18: now also U?.B18 (PS_MIO18_501)
- net B19: now also U?.B19 (IO_L2P_T0_AD8P_35)
- net B2: now also U?.B2 (PS_DDR_DQS_N0_502)
- net B20: now also U?.B20 (IO_L1N_T0_AD0N_35)
- net B3: now also U?.B3 (PS_DDR_DQ1_502)
- net B4: now also U?.B4 (PS_DDR_DRST_B_502)
- net B5: now also U?.B5 (PS_MIO9_500)
- net B6: now also U?.B6 (VCCO_MIO0_500)
- net B7: now also U?.B7 (PS_MIO4_500)
- net B8: now also U?.B8 (PS_MIO2_500)
- net B9: now also U?.B9 (PS_MIO51_501)
- net C1: now also U?.C1 (PS_DDR_DQ6_502)
- net C10: now also U?.C10 (PS_MIO52_501)
- net C11: now also U?.C11 (PS_MIO53_501)
- net C12: now also U?.C12 (PS_MIO49_501)
- net C13: now also U?.C13 (PS_MIO29_501)
- net C15: now also U?.C15 (PS_MIO30_501)
- net C16: now also U?.C16 (PS_MIO28_501)
- net C17: now also U?.C17 (PS_MIO41_501)
- net C18: now also U?.C18 (PS_MIO39_501)
- net C19: now also U?.C19 (VCCO_35)
- net C2: now also U?.C2 (PS_DDR_DQS_P0_502)
- net C20: now also U?.C20 (IO_L1P_T0_AD0P_35)
- net C3: now also U?.C3 (PS_DDR_DQ0_502)
- net C5: now also U?.C5 (PS_MIO14_500)
- net C6: now also U?.C6 (PS_MIO11_500)
- net C7: now also U?.C7 (PS_POR_B_500)
- net C8: now also U?.C8 (PS_MIO15_500)
- net D1: now also U?.D1 (PS_DDR_DQ5_502)
- net D10: now also U?.D10 (PS_MIO19_501)
- net D11: now also U?.D11 (PS_MIO23_501)
- net D13: now also U?.D13 (PS_MIO27_501)
- net D14: now also U?.D14 (PS_MIO40_501)
- net D15: now also U?.D15 (PS_MIO33_501)
- net D16: now also U?.D16 (PS_MIO46_501)
- net D18: now also U?.D18 (IO_L3N_T0_DQS_AD1N_35)
- net D19: now also U?.D19 (IO_L4P_T0_35)
- net D20: now also U?.D20 (IO_L4N_T0_35)
- net D3: now also U?.D3 (PS_DDR_DQ4_502)
- net D4: now also U?.D4 (PS_DDR_A13_502)
- net D5: now also U?.D5 (PS_MIO8_500)
- net D6: now also U?.D6 (PS_MIO3_500)
- net D8: now also U?.D8 (PS_MIO7_500)
- net D9: now also U?.D9 (PS_MIO12_500)
- net E1: now also U?.E1 (PS_DDR_DQ7_502)
- net E11: now also U?.E11 (PS_MIO_VREF_501)
- net E12: now also U?.E12 (PS_MIO42_501)
- net E13: now also U?.E13 (PS_MIO38_501)
- net E14: now also U?.E14 (PS_MIO17_501)
- net E16: now also U?.E16 (PS_MIO31_501)
- net E17: now also U?.E17 (IO_L3P_T0_DQS_AD1P_35)
- net E18: now also U?.E18 (IO_L5P_T0_AD9P_35)
- net E19: now also U?.E19 (IO_L5N_T0_AD9N_35)
- net E2: now also U?.E2 (PS_DDR_DQ8_502)
- net E3: now also U?.E3 (PS_DDR_DQ9_502)
- net E4: now also U?.E4 (PS_DDR_A12_502)
- net E6: now also U?.E6 (PS_MIO0_500)
- net E7: now also U?.E7 (PS_CLK_500)
- net E8: now also U?.E8 (PS_MIO13_500)
- net E9: now also U?.E9 (PS_MIO10_500)
- net F1: now also U?.F1 (PS_DDR_DM1_502)
- net F10: now also U?.F10 (RSVDGND)
- net F11: now also U?.F11 (VCCBATT_0)
- net F12: now also U?.F12 (PS_MIO35_501)
- net F13: now also U?.F13 (PS_MIO44_501)
- net F14: now also U?.F14 (PS_MIO21_501)
- net F15: now also U?.F15 (PS_MIO25_501)
- net F16: now also U?.F16 (IO_L6P_T0_35)
- net F17: now also U?.F17 (IO_L6N_T0_VREF_35)
- net F19: now also U?.F19 (IO_L15P_T2_DQS_AD12P_35)
- net F2: now also U?.F2 (PS_DDR_DQS_N1_502)
- net F20: now also U?.F20 (IO_L15N_T2_DQS_AD12N_35)
- net F4: now also U?.F4 (PS_DDR_A14_502)
- net F5: now also U?.F5 (PS_DDR_A10_502)
- net F6: now also U?.F6 (TDO_0)
- net F9: now also U?.F9 (TCK_0)
- net G11: now also U?.G11 (VCCBRAM)
- net G13: now also U?.G13 (VCCINT)
- net G14: now also U?.G14 (IO_0_35)
- net G15: now also U?.G15 (IO_L19N_T3_VREF_35)
- net G17: now also U?.G17 (IO_L16P_T2_35)
- net G18: now also U?.G18 (IO_L16N_T2_35)
- net G19: now also U?.G19 (IO_L18P_T2_AD13P_35)
- net G2: now also U?.G2 (PS_DDR_DQS_P1_502)
- net G20: now also U?.G20 (IO_L18N_T2_AD13N_35)
- net G3: now also U?.G3 (PS_DDR_DQ10_502)
- net G4: now also U?.G4 (PS_DDR_A11_502)
- net G5: now also U?.G5 (PS_DDR_VRN_502)
- net G6: now also U?.G6 (TDI_0)
- net G7: now also U?.G7 (VCCPINT)
- net G8: now also U?.G8 (VCCPLL)
- net G9: now also U?.G9 (VCCPAUX)
- net H1: now also U?.H1 (PS_DDR_DQ14_502)
- net H15: now also U?.H15 (IO_L19P_T3_35)
- net H16: now also U?.H16 (IO_L13P_T2_MRCC_35)
- net H17: now also U?.H17 (IO_L13N_T2_MRCC_35)
- net H18: now also U?.H18 (IO_L14N_T2_AD4N_SRCC_35)
- net H2: now also U?.H2 (PS_DDR_DQ13_502)
- net H20: now also U?.H20 (IO_L17N_T2_AD5N_35)
- net H3: now also U?.H3 (PS_DDR_DQ11_502)
- net H5: now also U?.H5 (PS_DDR_VRP_502)
- net H6: now also U?.H6 (PS_DDR_VREF0_502)
- net J1: now also U?.J1 (PS_DDR_DQ15_502)
- net J10: now also U?.J10 (GNDADC_0)
- net J11: now also U?.J11 (VCCAUX)
- net J14: now also U?.J14 (IO_L20N_T3_AD6N_35)
- net J15: now also U?.J15 (IO_25_35)
- net J16: now also U?.J16 (IO_L24N_T3_AD15N_35)
- net J18: now also U?.J18 (IO_L14P_T2_AD4P_SRCC_35)
- net J19: now also U?.J19 (IO_L10N_T1_AD11N_35)
- net J20: now also U?.J20 (IO_L17P_T2_AD5P_35)
- net J3: now also U?.J3 (PS_DDR_DQ12_502)
- net J4: now also U?.J4 (PS_DDR_A9_502)
- net J5: now also U?.J5 (PS_DDR_BA2_502)
- net J6: now also U?.J6 (TMS_0)
- net J9: now also U?.J9 (VCCADC_0)
- net K1: now also U?.K1 (PS_DDR_A8_502)
- net K10: now also U?.K10 (VREFN_0)
- net K14: now also U?.K14 (IO_L20P_T3_AD6P_35)
- net K16: now also U?.K16 (IO_L24P_T3_AD15P_35)
- net K17: now also U?.K17 (IO_L12P_T1_MRCC_35)
- net K18: now also U?.K18 (IO_L12N_T1_MRCC_35)
- net K19: now also U?.K19 (IO_L10P_T1_AD11P_35)
- net K2: now also U?.K2 (PS_DDR_A1_502)
- net K3: now also U?.K3 (PS_DDR_A3_502)
- net K4: now also U?.K4 (PS_DDR_A7_502)
- net K6: now also U?.K6 (VCCO_0)
- net K9: now also U?.K9 (VP_0)
- net L1: now also U?.L1 (PS_DDR_A5_502)
- net L10: now also U?.L10 (VN_0)
- net L14: now also U?.L14 (IO_L22P_T3_AD7P_35)
- net L15: now also U?.L15 (IO_L22N_T3_AD7N_35)
- net L16: now also U?.L16 (IO_L11P_T1_SRCC_35)
- net L17: now also U?.L17 (IO_L11N_T1_SRCC_35)
- net L19: now also U?.L19 (IO_L9P_T1_DQS_AD3P_35)
- net L2: now also U?.L2 (PS_DDR_CKP_502)
- net L20: now also U?.L20 (IO_L9N_T1_DQS_AD3N_35)
- net L4: now also U?.L4 (PS_DDR_A6_502)
- net L5: now also U?.L5 (PS_DDR_BA0_502)
- net L6: now also U?.L6 (PROGRAM_B_0)
- net L9: now also U?.L9 (VREFP_0)
- net M10: now also U?.M10 (DXN_0)
- net M14: now also U?.M14 (IO_L23P_T3_35)
- net M15: now also U?.M15 (IO_L23N_T3_35)
- net M17: now also U?.M17 (IO_L8P_T1_AD10P_35)
- net M18: now also U?.M18 (IO_L8N_T1_AD10N_35)
- net M19: now also U?.M19 (IO_L7P_T1_AD2P_35)
- net M2: now also U?.M2 (PS_DDR_CKN_502)
- net M20: now also U?.M20 (IO_L7N_T1_AD2N_35)
- net M3: now also U?.M3 (PS_DDR_A2_502)
- net M4: now also U?.M4 (PS_DDR_A4_502)
- net M5: now also U?.M5 (PS_DDR_WE_B_502)
- net M6: now also U?.M6 (CFGBVS_0)
- net M9: now also U?.M9 (DXP_0)
- net N1: now also U?.N1 (PS_DDR_CS_B_502)
- net N15: now also U?.N15 (IO_L21P_T3_DQS_AD14P_35)
- net N16: now also U?.N16 (IO_L21N_T3_DQS_AD14N_35)
- net N17: now also U?.N17 (IO_L23P_T3_34)
- net N18: now also U?.N18 (IO_L13P_T2_MRCC_34)
- net N19: now also U?.N19 (VCCO_34)
- net N2: now also U?.N2 (PS_DDR_A0_502)
- net N20: now also U?.N20 (IO_L14P_T2_SRCC_34)
- net N3: now also U?.N3 (PS_DDR_CKE_502)
- net N5: now also U?.N5 (PS_DDR_ODT_502)
- net N6: now also U?.N6 (RSVDVCC3)
- net P1: now also U?.P1 (PS_DDR_DQ16_502)
- net P14: now also U?.P14 (IO_L6P_T0_34)
- net P15: now also U?.P15 (IO_L24P_T3_34)
- net P16: now also U?.P16 (IO_L24N_T3_34)
- net P18: now also U?.P18 (IO_L23N_T3_34)
- net P19: now also U?.P19 (IO_L13N_T2_MRCC_34)
- net P20: now also U?.P20 (IO_L14N_T2_SRCC_34)
- net P3: now also U?.P3 (PS_DDR_DQ17_502)
- net P4: now also U?.P4 (PS_DDR_RAS_B_502)
- net P5: now also U?.P5 (PS_DDR_CAS_B_502)
- net P6: now also U?.P6 (PS_DDR_VREF1_502)
- net R1: now also U?.R1 (PS_DDR_DQ19_502)
- net R10: now also U?.R10 (INIT_B_0)
- net R11: now also U?.R11 (DONE_0)
- net R14: now also U?.R14 (IO_L6N_T0_VREF_34)
- net R16: now also U?.R16 (IO_L19P_T3_34)
- net R17: now also U?.R17 (IO_L19N_T3_VREF_34)
- net R18: now also U?.R18 (IO_L20N_T3_34)
- net R19: now also U?.R19 (IO_0_34)
- net R2: now also U?.R2 (PS_DDR_DQS_P2_502)
- net R3: now also U?.R3 (PS_DDR_DQ18_502)
- net R4: now also U?.R4 (PS_DDR_BA1_502)
- net R6: now also U?.R6 (RSVDVCC2)
- net T1: now also U?.T1 (PS_DDR_DM2_502)
- net T10: now also U?.T10 (IO_L1N_T0_34)
- net T11: now also U?.T11 (IO_L1P_T0_34)
- net T12: now also U?.T12 (IO_L2P_T0_34)
- net T14: now also U?.T14 (IO_L5P_T0_34)
- net T15: now also U?.T15 (IO_L5N_T0_34)
- net T16: now also U?.T16 (IO_L9P_T1_DQS_34)
- net T17: now also U?.T17 (IO_L20P_T3_34)
- net T19: now also U?.T19 (IO_25_34)
- net T2: now also U?.T2 (PS_DDR_DQS_N2_502)
- net T20: now also U?.T20 (IO_L15P_T2_DQS_34)
- net T4: now also U?.T4 (PS_DDR_DQ20_502)
- net T6: now also U?.T6 (RSVDVCC1)
- net T8: now also U?.T8 (VCCO_13)
- net U12: now also U?.U12 (IO_L2N_T0_34)
- net U13: now also U?.U13 (IO_L3P_T0_DQS_PUDC_B_34)
- net U14: now also U?.U14 (IO_L11P_T1_SRCC_34)
- net U15: now also U?.U15 (IO_L11N_T1_SRCC_34)
- net U17: now also U?.U17 (IO_L9N_T1_DQS_34)
- net U18: now also U?.U18 (IO_L12P_T1_MRCC_34)
- net U19: now also U?.U19 (IO_L12N_T1_MRCC_34)
- net U2: now also U?.U2 (PS_DDR_DQ22_502)
- net U20: now also U?.U20 (IO_L15N_T2_DQS_34)
- net U3: now also U?.U3 (PS_DDR_DQ23_502)
- net U4: now also U?.U4 (PS_DDR_DQ21_502)
- net V1: now also U?.V1 (PS_DDR_DQ24_502)
- net V12: now also U?.V12 (IO_L4P_T0_34)
- net V13: now also U?.V13 (IO_L3N_T0_DQS_34)
- net V15: now also U?.V15 (IO_L10P_T1_34)
- net V16: now also U?.V16 (IO_L18P_T2_34)
- net V17: now also U?.V17 (IO_L21P_T3_DQS_34)
- net V18: now also U?.V18 (IO_L21N_T3_DQS_34)
- net V2: now also U?.V2 (PS_DDR_DQ30_502)
- net V20: now also U?.V20 (IO_L16P_T2_34)
- net V3: now also U?.V3 (PS_DDR_DQ31_502)
- net W1: now also U?.W1 (PS_DDR_DQ26_502)
- net W13: now also U?.W13 (IO_L4N_T0_34)
- net W14: now also U?.W14 (IO_L8P_T1_34)
- net W15: now also U?.W15 (IO_L10N_T1_34)
- net W16: now also U?.W16 (IO_L18N_T2_34)
- net W18: now also U?.W18 (IO_L22P_T3_34)
- net W19: now also U?.W19 (IO_L22N_T3_34)
- net W20: now also U?.W20 (IO_L16N_T2_34)
- net W3: now also U?.W3 (PS_DDR_DQ29_502)
- net W4: now also U?.W4 (PS_DDR_DQS_N3_502)
- net W5: now also U?.W5 (PS_DDR_DQS_P3_502)
- net Y1: now also U?.Y1 (PS_DDR_DM3_502)
- net Y14: now also U?.Y14 (IO_L8N_T1_34)
- net Y16: now also U?.Y16 (IO_L7P_T1_34)
- net Y17: now also U?.Y17 (IO_L7N_T1_34)
- net Y18: now also U?.Y18 (IO_L17P_T2_34)
- net Y19: now also U?.Y19 (IO_L17N_T2_34)
- net Y2: now also U?.Y2 (PS_DDR_DQ28_502)
- net Y3: now also U?.Y3 (PS_DDR_DQ25_502)
- net Y4: now also U?.Y4 (PS_DDR_DQ27_502)
- new net A18: U?.A18 (GND)
- new net B1: U?.B1 (GND)
- new net B11: U?.B11 (GND)
- new net B16: U?.B16 (VCCO_MIO1_501)
- new net C14: U?.C14 (GND)
- new net C4: U?.C4 (GND)
- new net C9: U?.C9 (GND)
- new net D12: U?.D12 (VCCO_MIO1_501)
- new net D17: U?.D17 (GND)
- new net D2: U?.D2 (VCCO_DDR_502)
- new net D7: U?.D7 (VCCO_MIO0_500)
- new net E10: U?.E10 (GND)
- new net E15: U?.E15 (VCCO_MIO1_501)
- new net E20: U?.E20 (GND)
- new net E5: U?.E5 (VCCO_DDR_502)
- new net F18: U?.F18 (VCCO_35)
- new net F3: U?.F3 (GND)
- new net F7: U?.F7 (GND)
- new net F8: U?.F8 (VCCPAUX)
- new net G1: U?.G1 (VCCO_DDR_502)
- new net G10: U?.G10 (GND)
- new net G12: U?.G12 (GND)
- new net G16: U?.G16 (GND)
- new net H10: U?.H10 (VCCBRAM)
- new net H11: U?.H11 (GND)
- new net H12: U?.H12 (VCCINT)
- new net H13: U?.H13 (GND)
- new net H14: U?.H14 (VCCO_35)
- new net H19: U?.H19 (GND)
- new net H4: U?.H4 (VCCO_DDR_502)
- new net H7: U?.H7 (GND)
- new net H8: U?.H8 (VCCPAUX)
- new net H9: U?.H9 (GND)
- new net J12: U?.J12 (GND)
- new net J13: U?.J13 (VCCINT)
- new net J17: U?.J17 (VCCO_35)
- new net J2: U?.J2 (GND)
- new net J7: U?.J7 (VCCPINT)
- new net J8: U?.J8 (GND)
- new net K11: U?.K11 (GND)
- new net K12: U?.K12 (VCCINT)
- new net K13: U?.K13 (GND)
- new net K15: U?.K15 (GND)
- new net K20: U?.K20 (VCCO_35)
- new net K5: U?.K5 (GND)
- new net K7: U?.K7 (GND)
- new net K8: U?.K8 (VCCPAUX)
- new net L11: U?.L11 (VCCAUX)
- new net L12: U?.L12 (GND)
- new net L13: U?.L13 (VCCINT)
- new net L18: U?.L18 (GND)
- new net L3: U?.L3 (VCCO_DDR_502)
- new net L7: U?.L7 (VCCPINT)
- new net L8: U?.L8 (GND)
- new net M1: U?.M1 (GND)
- new net M11: U?.M11 (GND)
- new net M12: U?.M12 (VCCINT)
- new net M13: U?.M13 (GND)
- new net M16: U?.M16 (VCCO_35)
- new net M7: U?.M7 (GND)
- new net M8: U?.M8 (VCCPAUX)
- new net N10: U?.N10 (GND)
- new net N11: U?.N11 (VCCAUX)
- new net N12: U?.N12 (GND)
- new net N13: U?.N13 (VCCINT)
- new net N14: U?.N14 (GND)
- new net N4: U?.N4 (GND)
- new net N7: U?.N7 (VCCPINT)
- new net N8: U?.N8 (GND)
- new net N9: U?.N9 (VCCAUX)
- new net P10: U?.P10 (VCCAUX)
- new net P11: U?.P11 (GND)
- new net P12: U?.P12 (VCCINT)
- new net P13: U?.P13 (GND)
- new net P17: U?.P17 (GND)
- new net P2: U?.P2 (VCCO_DDR_502)
- new net P7: U?.P7 (GND)
- new net P8: U?.P8 (VCCPINT)
- new net P9: U?.P9 (GND)
- new net R12: U?.R12 (GND)
- new net R13: U?.R13 (VCCINT)
- new net R15: U?.R15 (VCCO_34)
- new net R20: U?.R20 (GND)
- new net R5: U?.R5 (VCCO_DDR_502)
- new net R7: U?.R7 (VCCPINT)
- new net R8: U?.R8 (GND)
- new net R9: U?.R9 (VCCAUX)
- new net T13: U?.T13 (GND)
- new net T18: U?.T18 (VCCO_34)
- new net T3: U?.T3 (GND)
- new net T5: U?.T5 (NC)
- new net T7: U?.T7 (GND)
- new net T9: U?.T9 (NC)
- new net U1: U?.U1 (VCCO_DDR_502)
- new net U10: U?.U10 (NC)
- new net U11: U?.U11 (VCCO_13)
- new net U16: U?.U16 (GND)
- new net U5: U?.U5 (NC)
- new net U6: U?.U6 (GND)
- new net U7: U?.U7 (NC)
- new net U8: U?.U8 (NC)
- new net U9: U?.U9 (NC)
- new net V10: U?.V10 (NC)
- new net V11: U?.V11 (NC)
- new net V14: U?.V14 (VCCO_34)
- new net V19: U?.V19 (GND)
- new net V4: U?.V4 (VCCO_DDR_502)
- new net V5: U?.V5 (NC)
- new net V6: U?.V6 (NC)
- new net V7: U?.V7 (NC)
- new net V8: U?.V8 (NC)
- new net V9: U?.V9 (GND)
- new net W10: U?.W10 (NC)
- new net W11: U?.W11 (NC)
- new net W12: U?.W12 (GND)
- new net W17: U?.W17 (VCCO_34)
- new net W2: U?.W2 (GND)
- new net W6: U?.W6 (NC)
- new net W7: U?.W7 (VCCO_13)
- new net W8: U?.W8 (NC)
- new net W9: U?.W9 (NC)
- new net Y10: U?.Y10 (VCCO_13)
- new net Y11: U?.Y11 (NC)
- new net Y12: U?.Y12 (NC)
- new net Y13: U?.Y13 (NC)
- new net Y15: U?.Y15 (GND)
- new net Y20: U?.Y20 (VCCO_34)
- new net Y5: U?.Y5 (GND)
- new net Y6: U?.Y6 (NC)
- new net Y7: U?.Y7 (NC)
- new net Y8: U?.Y8 (NC)
- new net Y9: U?.Y9 (NC)
