File: ebaz4205/components/xc7z010.kicad_sch (KiCad schematic)
At the start: 9 parts

Commit message: Consolidated all custom symbols into single library.
Library is available at ebaz4205/components/ebaz4205.kicad_sym

The templates and the schematics have been updated to use this library.
Keeping the original libraries for future reference.
Parts:
- removed U? (x9): xc7z010clg400, symbol xilinx7:xc7z010clg400
- added U? (x9): xc7z010clg400, symbol ebaz4205:xc7z010clg400
Connections:
- net A1: now also U?.A1 (PS_DDR_DM0_502)
- net A10: now also U?.A10 (PS_MIO37_501)
- net A11: now also U?.A11 (PS_MIO36_501)
- net A12: now also U?.A12 (PS_MIO34_501)
- net A13: now also U?.A13 (VCCO_MIO1_501)
- net A14: now also U?.A14 (PS_MIO32_501)
- net A15: now also U?.A15 (PS_MIO26_501)
- net A16: now also U?.A16 (PS_MIO24_501)
- net A17: now also U?.A17 (PS_MIO20_501)
- net A18: now also U?.A18 (GND)
- net A19: now also U?.A19 (PS_MIO16_501)
- net A2: now also U?.A2 (PS_DDR_DQ2_502)
- net A20: now also U?.A20 (IO_L2N_T0_AD8N_35)
- net A3: now also U?.A3 (VCCO_DDR_502)
- net A4: now also U?.A4 (PS_DDR_DQ3_502)
- net A5: now also U?.A5 (PS_MIO6_500)
- net A6: now also U?.A6 (PS_MIO5_500)
- net A7: now also U?.A7 (PS_MIO1_500)
- net A8: now also U?.A8 (GND)
- net A9: now also U?.A9 (PS_MIO43_501)
- net B1: now also U?.B1 (GND)
- net B10: now also U?.B10 (PS_SRST_B_501)
- net B11: now also U?.B11 (GND)
- net B12: now also U?.B12 (PS_MIO48_501)
- net B13: now also U?.B13 (PS_MIO50_501)
- net B14: now also U?.B14 (PS_MIO47_501)
- net B15: now also U?.B15 (PS_MIO45_501)
- net B16: now also U?.B16 (VCCO_MIO1_501)
- net B17: now also U?.B17 (PS_MIO22_501)
- net B18: now also U?.B18 (PS_MIO18_501)
- net B19: now also U?.B19 (IO_L2P_T0_AD8P_35)
- net B2: now also U?.B2 (PS_DDR_DQS_N0_502)
- net B20: now also U?.B20 (IO_L1N_T0_AD0N_35)
- net B3: now also U?.B3 (PS_DDR_DQ1_502)
- net B4: now also U?.B4 (PS_DDR_DRST_B_502)
- net B5: now also U?.B5 (PS_MIO9_500)
- net B6: now also U?.B6 (VCCO_MIO0_500)
- net B7: now also U?.B7 (PS_MIO4_500)
- net B8: now also U?.B8 (PS_MIO2_500)
- net B9: now also U?.B9 (PS_MIO51_501)
- net C1: now also U?.C1 (PS_DDR_DQ6_502)
- net C10: now also U?.C10 (PS_MIO52_501)
- net C11: now also U?.C11 (PS_MIO53_501)
- net C12: now also U?.C12 (PS_MIO49_501)
- net C13: now also U?.C13 (PS_MIO29_501)
- net C14: now also U?.C14 (GND)
- net C15: now also U?.C15 (PS_MIO30_501)
- net C16: now also U?.C16 (PS_MIO28_501)
- net C17: now also U?.C17 (PS_MIO41_501)
- net C18: now also U?.C18 (PS_MIO39_501)
- net C19: now also U?.C19 (VCCO_35)
- net C2: now also U?.C2 (PS_DDR_DQS_P0_502)
- net C20: now also U?.C20 (IO_L1P_T0_AD0P_35)
- net C3: now also U?.C3 (PS_DDR_DQ0_502)
- net C4: now also U?.C4 (GND)
- net C5: now also U?.C5 (PS_MIO14_500)
- net C6: now also U?.C6 (PS_MIO11_500)
- net C7: now also U?.C7 (PS_POR_B_500)
- net C8: now also U?.C8 (PS_MIO15_500)
- net C9: now also U?.C9 (GND)
- net D1: now also U?.D1 (PS_DDR_DQ5_502)
- net D10: now also U?.D10 (PS_MIO19_501)
- net D11: now also U?.D11 (PS_MIO23_501)
- net D12: now also U?.D12 (VCCO_MIO1_501)
- net D13: now also U?.D13 (PS_MIO27_501)
- net D14: now also U?.D14 (PS_MIO40_501)
- net D15: now also U?.D15 (PS_MIO33_501)
- net D16: now also U?.D16 (PS_MIO46_501)
- net D17: now also U?.D17 (GND)
- net D18: now also U?.D18 (IO_L3N_T0_DQS_AD1N_35)
- net D19: now also U?.D19 (IO_L4P_T0_35)
- net D2: now also U?.D2 (VCCO_DDR_502)
- net D20: now also U?.D20 (IO_L4N_T0_35)
- net D3: now also U?.D3 (PS_DDR_DQ4_502)
- net D4: now also U?.D4 (PS_DDR_A13_502)
- net D5: now also U?.D5 (PS_MIO8_500)
- net D6: now also U?.D6 (PS_MIO3_500)
- net D7: now also U?.D7 (VCCO_MIO0_500)
- net D8: now also U?.D8 (PS_MIO7_500)
- net D9: now also U?.D9 (PS_MIO12_500)
- net E1: now also U?.E1 (PS_DDR_DQ7_502)
- net E10: now also U?.E10 (GND)
- net E11: now also U?.E11 (PS_MIO_VREF_501)
- net E12: now also U?.E12 (PS_MIO42_501)
- net E13: now also U?.E13 (PS_MIO38_501)
- net E14: now also U?.E14 (PS_MIO17_501)
- net E15: now also U?.E15 (VCCO_MIO1_501)
- net E16: now also U?.E16 (PS_MIO31_501)
- net E17: now also U?.E17 (IO_L3P_T0_DQS_AD1P_35)
- net E18: now also U?.E18 (IO_L5P_T0_AD9P_35)
- net E19: now also U?.E19 (IO_L5N_T0_AD9N_35)
- net E2: now also U?.E2 (PS_DDR_DQ8_502)
- net E20: now also U?.E20 (GND)
- net E3: now also U?.E3 (PS_DDR_DQ9_502)
- net E4: now also U?.E4 (PS_DDR_A12_502)
- net E5: now also U?.E5 (VCCO_DDR_502)
- net E6: now also U?.E6 (PS_MIO0_500)
- net E7: now also U?.E7 (PS_CLK_500)
- net E8: now also U?.E8 (PS_MIO13_500)
- net E9: now also U?.E9 (PS_MIO10_500)
- net F1: now also U?.F1 (PS_DDR_DM1_502)
- net F10: now also U?.F10 (RSVDGND)
- net F11: now also U?.F11 (VCCBATT_0)
- net F12: now also U?.F12 (PS_MIO35_501)
- net F13: now also U?.F13 (PS_MIO44_501)
- net F14: now also U?.F14 (PS_MIO21_501)
- net F15: now also U?.F15 (PS_MIO25_501)
- net F16: now also U?.F16 (IO_L6P_T0_35)
- net F17: now also U?.F17 (IO_L6N_T0_VREF_35)
- net F18: now also U?.F18 (VCCO_35)
- net F19: now also U?.F19 (IO_L15P_T2_DQS_AD12P_35)
- net F2: now also U?.F2 (PS_DDR_DQS_N1_502)
- net F20: now also U?.F20 (IO_L15N_T2_DQS_AD12N_35)
- net F3: now also U?.F3 (GND)
- net F4: now also U?.F4 (PS_DDR_A14_502)
- net F5: now also U?.F5 (PS_DDR_A10_502)
- net F6: now also U?.F6 (TDO_0)
- net F7: now also U?.F7 (GND)
- net F8: now also U?.F8 (VCCPAUX)
- net F9: now also U?.F9 (TCK_0)
- net G1: now also U?.G1 (VCCO_DDR_502)
- net G10: now also U?.G10 (GND)
- net G11: now also U?.G11 (VCCBRAM)
- net G12: now also U?.G12 (GND)
- net G13: now also U?.G13 (VCCINT)
- net G14: now also U?.G14 (IO_0_35)
- net G15: now also U?.G15 (IO_L19N_T3_VREF_35)
- net G16: now also U?.G16 (GND)
- net G17: now also U?.G17 (IO_L16P_T2_35)
- net G18: now also U?.G18 (IO_L16N_T2_35)
- net G19: now also U?.G19 (IO_L18P_T2_AD13P_35)
- net G2: now also U?.G2 (PS_DDR_DQS_P1_502)
- net G20: now also U?.G20 (IO_L18N_T2_AD13N_35)
- net G3: now also U?.G3 (PS_DDR_DQ10_502)
- net G4: now also U?.G4 (PS_DDR_A11_502)
- net G5: now also U?.G5 (PS_DDR_VRN_502)
- net G6: now also U?.G6 (TDI_0)
- net G7: now also U?.G7 (VCCPINT)
- net G8: now also U?.G8 (VCCPLL)
- net G9: now also U?.G9 (VCCPAUX)
- net H1: now also U?.H1 (PS_DDR_DQ14_502)
- net H10: now also U?.H10 (VCCBRAM)
- net H11: now also U?.H11 (GND)
- net H12: now also U?.H12 (VCCINT)
- net H13: now also U?.H13 (GND)
- net H14: now also U?.H14 (VCCO_35)
- net H15: now also U?.H15 (IO_L19P_T3_35)
- net H16: now also U?.H16 (IO_L13P_T2_MRCC_35)
- net H17: now also U?.H17 (IO_L13N_T2_MRCC_35)
- net H18: now also U?.H18 (IO_L14N_T2_AD4N_SRCC_35)
- net H19: now also U?.H19 (GND)
- net H2: now also U?.H2 (PS_DDR_DQ13_502)
- net H20: now also U?.H20 (IO_L17N_T2_AD5N_35)
- net H3: now also U?.H3 (PS_DDR_DQ11_502)
- net H4: now also U?.H4 (VCCO_DDR_502)
- net H5: now also U?.H5 (PS_DDR_VRP_502)
- net H6: now also U?.H6 (PS_DDR_VREF0_502)
- net H7: now also U?.H7 (GND)
- net H8: now also U?.H8 (VCCPAUX)
- net H9: now also U?.H9 (GND)
- net J1: now also U?.J1 (PS_DDR_DQ15_502)
- net J10: now also U?.J10 (GNDADC_0)
- net J11: now also U?.J11 (VCCAUX)
- net J12: now also U?.J12 (GND)
- net J13: now also U?.J13 (VCCINT)
- net J14: now also U?.J14 (IO_L20N_T3_AD6N_35)
- net J15: now also U?.J15 (IO_25_35)
- net J16: now also U?.J16 (IO_L24N_T3_AD15N_35)
- net J17: now also U?.J17 (VCCO_35)
- net J18: now also U?.J18 (IO_L14P_T2_AD4P_SRCC_35)
- net J19: now also U?.J19 (IO_L10N_T1_AD11N_35)
- net J2: now also U?.J2 (GND)
- net J20: now also U?.J20 (IO_L17P_T2_AD5P_35)
- net J3: now also U?.J3 (PS_DDR_DQ12_502)
- net J4: now also U?.J4 (PS_DDR_A9_502)
- net J5: now also U?.J5 (PS_DDR_BA2_502)
- net J6: now also U?.J6 (TMS_0)
- net J7: now also U?.J7 (VCCPINT)
- net J8: now also U?.J8 (GND)
- net J9: now also U?.J9 (VCCADC_0)
- net K1: now also U?.K1 (PS_DDR_A8_502)
- net K10: now also U?.K10 (VREFN_0)
- net K11: now also U?.K11 (GND)
- net K12: now also U?.K12 (VCCINT)
- net K13: now also U?.K13 (GND)
- net K14: now also U?.K14 (IO_L20P_T3_AD6P_35)
- net K15: now also U?.K15 (GND)
- net K16: now also U?.K16 (IO_L24P_T3_AD15P_35)
- net K17: now also U?.K17 (IO_L12P_T1_MRCC_35)
- net K18: now also U?.K18 (IO_L12N_T1_MRCC_35)
- net K19: now also U?.K19 (IO_L10P_T1_AD11P_35)
- net K2: now also U?.K2 (PS_DDR_A1_502)
- net K20: now also U?.K20 (VCCO_35)
- net K3: now also U?.K3 (PS_DDR_A3_502)
- net K4: now also U?.K4 (PS_DDR_A7_502)
- net K5: now also U?.K5 (GND)
- net K6: now also U?.K6 (VCCO_0)
- net K7: now also U?.K7 (GND)
- net K8: now also U?.K8 (VCCPAUX)
- net K9: now also U?.K9 (VP_0)
- net L1: now also U?.L1 (PS_DDR_A5_502)
- net L10: now also U?.L10 (VN_0)
- net L11: now also U?.L11 (VCCAUX)
- net L12: now also U?.L12 (GND)
- net L13: now also U?.L13 (VCCINT)
- net L14: now also U?.L14 (IO_L22P_T3_AD7P_35)
- net L15: now also U?.L15 (IO_L22N_T3_AD7N_35)
- net L16: now also U?.L16 (IO_L11P_T1_SRCC_35)
- net L17: now also U?.L17 (IO_L11N_T1_SRCC_35)
- net L18: now also U?.L18 (GND)
- net L19: now also U?.L19 (IO_L9P_T1_DQS_AD3P_35)
- net L2: now also U?.L2 (PS_DDR_CKP_502)
- net L20: now also U?.L20 (IO_L9N_T1_DQS_AD3N_35)
- net L3: now also U?.L3 (VCCO_DDR_502)
- net L4: now also U?.L4 (PS_DDR_A6_502)
- net L5: now also U?.L5 (PS_DDR_BA0_502)
- net L6: now also U?.L6 (PROGRAM_B_0)
- net L7: now also U?.L7 (VCCPINT)
- net L8: now also U?.L8 (GND)
- net L9: now also U?.L9 (VREFP_0)
- net M1: now also U?.M1 (GND)
- net M10: now also U?.M10 (DXN_0)
- net M11: now also U?.M11 (GND)
- net M12: now also U?.M12 (VCCINT)
- net M13: now also U?.M13 (GND)
- net M14: now also U?.M14 (IO_L23P_T3_35)
- net M15: now also U?.M15 (IO_L23N_T3_35)
- net M16: now also U?.M16 (VCCO_35)
- net M17: now also U?.M17 (IO_L8P_T1_AD10P_35)
- net M18: now also U?.M18 (IO_L8N_T1_AD10N_35)
- net M19: now also U?.M19 (IO_L7P_T1_AD2P_35)
- net M2: now also U?.M2 (PS_DDR_CKN_502)
- net M20: now also U?.M20 (IO_L7N_T1_AD2N_35)
- net M3: now also U?.M3 (PS_DDR_A2_502)
- net M4: now also U?.M4 (PS_DDR_A4_502)
- net M5: now also U?.M5 (PS_DDR_WE_B_502)
- net M6: now also U?.M6 (CFGBVS_0)
- net M7: now also U?.M7 (GND)
- net M8: now also U?.M8 (VCCPAUX)
- net M9: now also U?.M9 (DXP_0)
- net N1: now also U?.N1 (PS_DDR_CS_B_502)
- net N10: now also U?.N10 (GND)
- net N11: now also U?.N11 (VCCAUX)
- net N12: now also U?.N12 (GND)
- net N13: now also U?.N13 (VCCINT)
- net N14: now also U?.N14 (GND)
- net N15: now also U?.N15 (IO_L21P_T3_DQS_AD14P_35)
- net N16: now also U?.N16 (IO_L21N_T3_DQS_AD14N_35)
- net N17: now also U?.N17 (IO_L23P_T3_34)
- net N18: now also U?.N18 (IO_L13P_T2_MRCC_34)
- net N19: now also U?.N19 (VCCO_34)
- net N2: now also U?.N2 (PS_DDR_A0_502)
- net N20: now also U?.N20 (IO_L14P_T2_SRCC_34)
- net N3: now also U?.N3 (PS_DDR_CKE_502)
- net N4: now also U?.N4 (GND)
- net N5: now also U?.N5 (PS_DDR_ODT_502)
- net N6: now also U?.N6 (RSVDVCC3)
- net N7: now also U?.N7 (VCCPINT)
- net N8: now also U?.N8 (GND)
- net N9: now also U?.N9 (VCCAUX)
- net P1: now also U?.P1 (PS_DDR_DQ16_502)
- net P10: now also U?.P10 (VCCAUX)
- net P11: now also U?.P11 (GND)
- net P12: now also U?.P12 (VCCINT)
- net P13: now also U?.P13 (GND)
- net P14: now also U?.P14 (IO_L6P_T0_34)
- net P15: now also U?.P15 (IO_L24P_T3_34)
- net P16: now also U?.P16 (IO_L24N_T3_34)
- net P17: now also U?.P17 (GND)
- net P18: now also U?.P18 (IO_L23N_T3_34)
- net P19: now also U?.P19 (IO_L13N_T2_MRCC_34)
- net P2: now also U?.P2 (VCCO_DDR_502)
- net P20: now also U?.P20 (IO_L14N_T2_SRCC_34)
- net P3: now also U?.P3 (PS_DDR_DQ17_502)
- net P4: now also U?.P4 (PS_DDR_RAS_B_502)
- net P5: now also U?.P5 (PS_DDR_CAS_B_502)
- net P6: now also U?.P6 (PS_DDR_VREF1_502)
- net P7: now also U?.P7 (GND)
- net P8: now also U?.P8 (VCCPINT)
- net P9: now also U?.P9 (GND)
- net R1: now also U?.R1 (PS_DDR_DQ19_502)
- net R10: now also U?.R10 (INIT_B_0)
- net R11: now also U?.R11 (DONE_0)
- net R12: now also U?.R12 (GND)
- net R13: now also U?.R13 (VCCINT)
- net R14: now also U?.R14 (IO_L6N_T0_VREF_34)
- net R15: now also U?.R15 (VCCO_34)
- net R16: now also U?.R16 (IO_L19P_T3_34)
- net R17: now also U?.R17 (IO_L19N_T3_VREF_34)
- net R18: now also U?.R18 (IO_L20N_T3_34)
- net R19: now also U?.R19 (IO_0_34)
- net R2: now also U?.R2 (PS_DDR_DQS_P2_502)
- net R20: now also U?.R20 (GND)
- net R3: now also U?.R3 (PS_DDR_DQ18_502)
- net R4: now also U?.R4 (PS_DDR_BA1_502)
- net R5: now also U?.R5 (VCCO_DDR_502)
- net R6: now also U?.R6 (RSVDVCC2)
- net R7: now also U?.R7 (VCCPINT)
- net R8: now also U?.R8 (GND)
- net R9: now also U?.R9 (VCCAUX)
- net T1: now also U?.T1 (PS_DDR_DM2_502)
- net T10: now also U?.T10 (IO_L1N_T0_34)
- net T11: now also U?.T11 (IO_L1P_T0_34)
- net T12: now also U?.T12 (IO_L2P_T0_34)
- net T13: now also U?.T13 (GND)
- net T14: now also U?.T14 (IO_L5P_T0_34)
- net T15: now also U?.T15 (IO_L5N_T0_34)
- net T16: now also U?.T16 (IO_L9P_T1_DQS_34)
- net T17: now also U?.T17 (IO_L20P_T3_34)
- net T18: now also U?.T18 (VCCO_34)
- net T19: now also U?.T19 (IO_25_34)
- net T2: now also U?.T2 (PS_DDR_DQS_N2_502)
- net T20: now also U?.T20 (IO_L15P_T2_DQS_34)
- net T3: now also U?.T3 (GND)
- net T4: now also U?.T4 (PS_DDR_DQ20_502)
- net T5: now also U?.T5 (NC)
- net T6: now also U?.T6 (RSVDVCC1)
- net T7: now also U?.T7 (GND)
- net T8: now also U?.T8 (VCCO_13)
- net T9: now also U?.T9 (NC)
- net U1: now also U?.U1 (VCCO_DDR_502)
- net U10: now also U?.U10 (NC)
- net U11: now also U?.U11 (VCCO_13)
- net U12: now also U?.U12 (IO_L2N_T0_34)
- net U13: now also U?.U13 (IO_L3P_T0_DQS_PUDC_B_34)
- net U14: now also U?.U14 (IO_L11P_T1_SRCC_34)
- net U15: now also U?.U15 (IO_L11N_T1_SRCC_34)
- net U16: now also U?.U16 (GND)
- net U17: now also U?.U17 (IO_L9N_T1_DQS_34)
- net U18: now also U?.U18 (IO_L12P_T1_MRCC_34)
- net U19: now also U?.U19 (IO_L12N_T1_MRCC_34)
- net U2: now also U?.U2 (PS_DDR_DQ22_502)
- net U20: now also U?.U20 (IO_L15N_T2_DQS_34)
- net U3: now also U?.U3 (PS_DDR_DQ23_502)
- net U4: now also U?.U4 (PS_DDR_DQ21_502)
- net U5: now also U?.U5 (NC)
- net U6: now also U?.U6 (GND)
- net U7: now also U?.U7 (NC)
- net U8: now also U?.U8 (NC)
- net U9: now also U?.U9 (NC)
- net V1: now also U?.V1 (PS_DDR_DQ24_502)
- net V10: now also U?.V10 (NC)
- net V11: now also U?.V11 (NC)
- net V12: now also U?.V12 (IO_L4P_T0_34)
- net V13: now also U?.V13 (IO_L3N_T0_DQS_34)
- net V14: now also U?.V14 (VCCO_34)
- net V15: now also U?.V15 (IO_L10P_T1_34)
- net V16: now also U?.V16 (IO_L18P_T2_34)
- net V17: now also U?.V17 (IO_L21P_T3_DQS_34)
- net V18: now also U?.V18 (IO_L21N_T3_DQS_34)
- net V19: now also U?.V19 (GND)
- net V2: now also U?.V2 (PS_DDR_DQ30_502)
- net V20: now also U?.V20 (IO_L16P_T2_34)
- net V3: now also U?.V3 (PS_DDR_DQ31_502)
- net V4: now also U?.V4 (VCCO_DDR_502)
- net V5: now also U?.V5 (NC)
- net V6: now also U?.V6 (NC)
- net V7: now also U?.V7 (NC)
- net V8: now also U?.V8 (NC)
- net V9: now also U?.V9 (GND)
- net W1: now also U?.W1 (PS_DDR_DQ26_502)
- net W10: now also U?.W10 (NC)
- net W11: now also U?.W11 (NC)
- net W12: now also U?.W12 (GND)
- net W13: now also U?.W13 (IO_L4N_T0_34)
- net W14: now also U?.W14 (IO_L8P_T1_34)
- net W15: now also U?.W15 (IO_L10N_T1_34)
- net W16: now also U?.W16 (IO_L18N_T2_34)
- net W17: now also U?.W17 (VCCO_34)
- net W18: now also U?.W18 (IO_L22P_T3_34)
- net W19: now also U?.W19 (IO_L22N_T3_34)
- net W2: now also U?.W2 (GND)
- net W20: now also U?.W20 (IO_L16N_T2_34)
- net W3: now also U?.W3 (PS_DDR_DQ29_502)
- net W4: now also U?.W4 (PS_DDR_DQS_N3_502)
- net W5: now also U?.W5 (PS_DDR_DQS_P3_502)
- net W6: now also U?.W6 (NC)
- net W7: now also U?.W7 (VCCO_13)
- net W8: now also U?.W8 (NC)
- net W9: now also U?.W9 (NC)
- net Y1: now also U?.Y1 (PS_DDR_DM3_502)
- net Y10: now also U?.Y10 (VCCO_13)
- net Y11: now also U?.Y11 (NC)
- net Y12: now also U?.Y12 (NC)
- net Y13: now also U?.Y13 (NC)
- net Y14: now also U?.Y14 (IO_L8N_T1_34)
- net Y15: now also U?.Y15 (GND)
- net Y16: now also U?.Y16 (IO_L7P_T1_34)
- net Y17: now also U?.Y17 (IO_L7N_T1_34)
- net Y18: now also U?.Y18 (IO_L17P_T2_34)
- net Y19: now also U?.Y19 (IO_L17N_T2_34)
- net Y2: now also U?.Y2 (PS_DDR_DQ28_502)
- net Y20: now also U?.Y20 (VCCO_34)
- net Y3: now also U?.Y3 (PS_DDR_DQ25_502)
- net Y4: now also U?.Y4 (PS_DDR_DQ27_502)
- net Y5: now also U?.Y5 (GND)
- net Y6: now also U?.Y6 (NC)
- net Y7: now also U?.Y7 (NC)
- net Y8: now also U?.Y8 (NC)
- net Y9: now also U?.Y9 (NC)
Changed lines of the file:
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@@
     (effects (font (size 1.27 1.27)) (justify right))
   )
-  (symbol (lib_name "xilinx7:xc7z010clg400_2") (lib_id "xilinx7:xc7z010clg400") (at 54.61 8.89 0) (unit 2)
+  (symbol (lib_id "ebaz4205:xc7z010clg400") (at 54.61 8.89 0) (unit 2)
     (in_bom yes) (on_board yes)
     (property "Reference" "U?" (id 0) (at 59.69 2.54 0)
@@
     )
   )
-  (symbol (lib_name "xilinx7:xc7z010clg400_9") (lib_id "xilinx7:xc7z010clg400") (at 425.45 8.89 0) (unit 9)
+  (symbol (lib_id "ebaz4205:xc7z010clg400") (at 425.45 8.89 0) (unit 9)
     (in_bom yes) (on_board yes)
     (property "Reference" "U?" (id 0) (at 430.53 2.54 0)
@@
     )
   )
-  (symbol (lib_name "xilinx7:xc7z010clg400_1") (lib_id "xilinx7:xc7z010clg400") (at 16.51 8.89 0) (unit 1)
+  (symbol (lib_id "ebaz4205:xc7z010clg400") (at 16.51 8.89 0) (unit 1)
     (in_bom yes) (on_board yes)
     (property "Reference" "U?" (id 0) (at 21.59 2.54 0)
@@
     )
   )
-  (symbol (lib_name "xilinx7:xc7z010clg400_5") (lib_id "xilinx7:xc7z010clg400") (at 220.98 8.89 0) (unit 5)
+  (symbol (lib_id "ebaz4205:xc7z010clg400") (at 220.98 8.89 0) (unit 5)
     (in_bom yes) (on_board yes)
     (property "Reference" "U?" (id 0) (at 226.06 2.54 0)
@@
     )
   )
-  (symbol (lib_name "xilinx7:xc7z010clg400_6") (lib_id "xilinx7:xc7z010clg400") (at 274.32 8.89 0) (unit 6)
+  (symbol (lib_id "ebaz4205:xc7z010clg400") (at 274.32 8.89 0) (unit 6)
     (in_bom yes) (on_board yes)
     (property "Reference" "U?" (id 0) (at 279.4 2.54 0)
@@
     )
   )
-  (symbol (lib_name "xilinx7:xc7z010clg400_8") (lib_id "xilinx7:xc7z010clg400") (at 391.16 8.89 0) (unit 8)
+  (symbol (lib_id "ebaz4205:xc7z010clg400") (at 391.16 8.89 0) (unit 8)
     (in_bom yes) (on_board yes)
     (property "Reference" "U?" (id 0) (at 396.24 2.54 0)
@@
     )
   )
-  (symbol (lib_name "xilinx7:xc7z010clg400_3") (lib_id "xilinx7:xc7z010clg400") (at 92.71 8.89 0) (unit 3)
+  (symbol (lib_id "ebaz4205:xc7z010clg400") (at 92.71 8.89 0) (unit 3)
     (in_bom yes) (on_board yes)
     (property "Reference" "U?" (id 0) (at 97.79 2.54 0)
@@
     )
   )
-  (symbol (lib_name "xilinx7:xc7z010clg400_4") (lib_id "xilinx7:xc7z010clg400") (at 156.21 8.89 0) (unit 4)
+  (symbol (lib_id "ebaz4205:xc7z010clg400") (at 156.21 8.89 0) (unit 4)
     (in_bom yes) (on_board yes)
     (property "Reference" "U?" (id 0) (at 161.29 2.54 0)
@@
     )
   )
-  (symbol (lib_name "xilinx7:xc7z010clg400_7") (lib_id "xilinx7:xc7z010clg400") (at 331.47 8.89 0) (unit 7)
+  (symbol (lib_id "ebaz4205:xc7z010clg400") (at 331.47 8.89 0) (unit 7)
     (in_bom yes) (on_board yes)
     (property "Reference" "U?" (id 0) (at 336.55 2.54 0)
@@
   )
   (symbol_instances
-    (path "/0ad567ed-238b-4e80-b363-f8847fdf59fa"
+    (path "/c74f1e13-6f3a-4b0f-801c-7258c0069aaa"
       (reference "U?") (unit 1) (value "xc7z010clg400") (footprint "")
     )
-    (path "/b0fe23b2-d828-48d6-b868-b72c83488116"
+    (path "/4d001dc9-b5d3-4595-a30f-55d8337b5ff3"
       (reference "U?") (unit 2) (value "xc7z010clg400") (footprint "")
     )
-    (path "/b5e0bda7-2e9c-466e-a551-b90e0c93329c"
+    (path "/2a491273-0687-48cb-ad22-68732f416190"
       (reference "U?") (unit 3) (value "xc7z010clg400") (footprint "")
     )
-    (path "/96642803-ae26-4ce7-a846-80571229fb2a"
+    (path "/4d024a83-7367-4683-ac5a-bba0f53163c9"
       (reference "U?") (unit 4) (value "xc7z010clg400") (footprint "")
     )
-    (path "/3f46302f-d597-4535-b9c9-5237316abe20"
+    (path "/e234f092-ebe2-42dd-b071-d2fd5e7e186a"
       (reference "U?") (unit 5) (value "xc7z010clg400") (footprint "")
     )
-    (path "/0e2b711b-7565-4231-b20c-04a6a4c3a9d3"
+    (path "/27dde6ed-46ca-4ffc-8752-e457461183db"
       (reference "U?") (unit 6) (value "xc7z010clg400") (footprint "")
     )
-    (path "/1f83d365-9d24-4f0f-915f-8a003794a204"
+    (path "/e19b2676-cc36-4ad3-8ada-29261c7f19ef"
       (reference "U?") (unit 7) (value "xc7z010clg400") (footprint "")
     )
-    (path "/79794142-b24a-402a-b7cf-d2da259a1151"
+    (path "/c259c9d3-c2a7-481d-93e4-7506bea695b6"
       (reference "U?") (unit 8) (value "xc7z010clg400") (footprint "")
     )
-    (path "/e29fc92d-6d19-447f-96f2-d82b2ed76bb8"
+    (path "/9fe60bb2-d80c-4c52-8e10-f7c5f53d31df"
       (reference "U?") (unit 9) (value "xc7z010clg400") (footprint "")
     )
