File: ebaz4205/ebaz4205.kicad_sch (KiCad schematic)
At the start: 565 parts, among them J3 Conn_01x04, J4 Conn_02x03_Odd_Even, J5 Conn_01x04, J7 Conn_01x04, J8 Conn_02x07_Odd_Even, T6 HST-0041SAR, U12 W29N01HVSINA, U20 Q_NPN_BEC, U21 Q_NPN_BEC, U22 J37I, U23 U23, U24 IP101GA, U25 RJ45_LED, U26 J37I, U27 J37I, U28 J37I, U30 TPS3839DBZ, U31 xc7z010clg400, U65 SGM706, U66 MT41K128M16JT-125_AITK, U67 SFH617A-1, U68 SFH617A-1, U69 SFH617A-1, U7 Micro_SD_Card_mount, U70 SFH617A-1, U72 TPS51200AQDRCRQ1, X3 DS1307Z+, X5 TXC-EBAZ, X8 TXC-7C, Y2 RTC_XTAL, Y3 Crystal

Commit message: Provided the resulting schematic.
Parts:
- removed LED6: LED_ALT, symbol Device:LED_ALT
- added LED6: LED_dual, symbol led:LED_dual
Connections:
- net GND: now also U24.40 (NC)
- net NetLED6_1: now also LED6.1 (A1)
- net NetLED6_2: now also LED6.2 (A2)
- net NetU24_15: now also U24.15 (NC)
- net REGOUT.0: now also U24.32 (NC)
- net U3.W13_0: now also LED6.4 (K1)
- net U3.W14_0: now also LED6.3 (K2)
- net VCC: now also U24.41 (NC), U24.44 (NC)

Commit message: Consolidated all custom symbols into single library.
Library is available at ebaz4205/components/ebaz4205.kicad_sym

The templates and the schematics have been updated to use this library.
Keeping the original libraries for future reference.
Parts:
- removed LED6: LED_dual, symbol led:LED_dual
- removed T6: HST-0041SAR, symbol trafo:HST-0041SAR
- removed U12: W29N01HVSINA, SOP50P2000X120-48N, symbol W29N01HVSINA:W29N01HVSINA
- removed U22, U26, U27, U28: J37I, symbol dcdc:J37I
- removed U23: U23, symbol unknown:U23
- removed U24: IP101GA, symbol eth:IP101GA
- removed U25: RJ45_LED, symbol Connector:RJ45_LED
- removed U30: TPS3839DBZ, Package_TO_SOT_SMD:SOT-23, symbol Power_Supervisor:TPS3839DBZ
- removed U31: xc7z010clg400, symbol xilinx7:xc7z010clg400
- removed U65: SGM706, symbol supervisor:SGM706
- removed U66: MT41K128M16JT-125_AITK, Micron-JT-0-0-*, symbol eec:MT41K128M16JT-125_AITK
- removed U67, U68, U69, U70: SFH617A-1, Package_DIP:DIP-4_W7.62mm, symbol Isolator:SFH617A-1
- removed U7: Micro_SD_Card_mount, symbol sd_card:Micro_SD_Card_mount
- removed U72: TPS51200AQDRCRQ1, TPS51200AQDRCRQ1, symbol TPS51200AQDRCRQ1:TPS51200AQDRCRQ1
- removed X3: DS1307Z+, SOIC127P600X175-8N, symbol DS1307Z+:DS1307Z+
- removed X5: TXC-EBAZ, symbol osc:TXC-EBAZ
- removed X8: TXC-7C, Oscillator:Oscillator_SMD_TXC_7C-4Pin_5.0x3.2mm, symbol Oscillator:TXC-7C
- removed Y2: RTC_XTAL, symbol osc:RTC_XTAL
- added LED6: LED_dual, symbol ebaz4205:LED_dual
- added T6: HST-0041SAR, symbol ebaz4205:HST-0041SAR
- added U12: W29N01HVSINA, SOP50P2000X120-48N, symbol ebaz4205:W29N01HVSINA
- added U22, U26, U27, U28: J37I, symbol ebaz4205:J37I
- added U23: U23, symbol ebaz4205:U23
- added U24: IP101GA, symbol ebaz4205:IP101GA
- added U25: 8P8C_LED, symbol ebaz4205:8P8C_LED
- added U30: TPS3839DBZ, Package_TO_SOT_SMD:SOT-23, symbol ebaz4205:TPS3839DBZ
- added U31: xc7z010clg400, symbol ebaz4205:xc7z010clg400
- added U65: SGM706, symbol ebaz4205:SGM706
- added U66: MT41K128M16JT-125_AITK, Micron-JT-0-0-*, symbol ebaz4205:MT41K128M16JT-125_AITK
- added U67, U68, U69, U70: TLP785, Package_DIP:DIP-4_W7.62mm, symbol ebaz4205:TLP785
- added U7: Micro_SD_Card_mount, symbol ebaz4205:Micro_SD_Card_mount
- added U72: TPS51200AQDRCRQ1, TPS51200AQDRCRQ1, symbol ebaz4205:TPS51200AQDRCRQ1
- added X3: DS1307Z+, SOIC127P600X175-8N, symbol ebaz4205:DS1307Z+
- added X5: TXC-EBAZ, symbol ebaz4205:TXC-EBAZ
- added X8: TXC-7C, Oscillator:Oscillator_SMD_TXC_7C-4Pin_5.0x3.2mm, symbol ebaz4205:TXC-7C
- added Y2: RTC_XTAL, symbol ebaz4205:RTC_XTAL
Connections:
- net #CE_0: now also U12.9 (#CE), U31.E6 (PS_MIO0_500)
- net #RE_0: now also U12.8 (#RE), U31.D5 (PS_MIO8_500)
- net #WE_0: now also U12.18 (#WE), U31.D6 (PS_MIO3_500)
- net ALE_0: now also U12.17 (ALE), U31.B8 (PS_MIO2_500)
- net CLE_0: now also U12.16 (CLE), U31.D8 (PS_MIO7_500)
- net CLK_0: now also U31.E7 (PS_CLK_500)
- net DATA1-11_0: now also U31.H17 (IO_L13N_T2_MRCC_35)
- net DATA1-13_0: now also U31.D20 (IO_L4N_T0_35)
- net DATA1-14_0: now also U31.D18 (IO_L3N_T0_DQS_AD1N_35)
- net DATA1-15_0: now also U31.H18 (IO_L14N_T2_AD4N_SRCC_35)
- net DATA1-16_0: now also U31.D19 (IO_L4P_T0_35)
- net DATA1-17_0: now also U31.F20 (IO_L15N_T2_DQS_AD12N_35)
- net DATA1-18_0: now also U31.E19 (IO_L5N_T0_AD9N_35)
- net DATA1-19_0: now also U31.F19 (IO_L15P_T2_DQS_AD12P_35)
- net DATA1-20_0: now also U31.K17 (IO_L12P_T1_MRCC_35)
- net DATA1-5_0: now also U31.A20 (IO_L2N_T0_AD8N_35)
- net DATA1-6_0: now also U31.H16 (IO_L13P_T2_MRCC_35)
- net DATA1-7_0: now also U31.B19 (IO_L2P_T0_AD8P_35)
- net DATA1-8_0: now also U31.B20 (IO_L1N_T0_AD0N_35)
- net DATA1-9_0: now also U31.C20 (IO_L1P_T0_AD0P_35)
- net DATA2-11_0: now also U31.K18 (IO_L12N_T1_MRCC_35)
- net DATA2-13_0: now also U31.K19 (IO_L10P_T1_AD11P_35)
- net DATA2-14_0: now also U31.J20 (IO_L17P_T2_AD5P_35)
- net DATA2-15_0: now also U31.L16 (IO_L11P_T1_SRCC_35)
- net DATA2-16_0: now also U31.L19 (IO_L9P_T1_DQS_AD3P_35)
- net DATA2-17_0: now also U31.M18 (IO_L8N_T1_AD10N_35)
- net DATA2-18_0: now also U31.L20 (IO_L9N_T1_DQS_AD3N_35)
- net DATA2-19_0: now also U31.M20 (IO_L7N_T1_AD2N_35)
- net DATA2-20_0: now also U31.L17 (IO_L11N_T1_SRCC_35)
- net DATA2-5_0: now also U31.G20 (IO_L18N_T2_AD13N_35)
- net DATA2-6_0: now also U31.J18 (IO_L14P_T2_AD4P_SRCC_35)
- net DATA2-7_0: now also U31.G19 (IO_L18P_T2_AD13P_35)
- net DATA2-8_0: now also U31.H20 (IO_L17N_T2_AD5N_35)
- net DATA2-9_0: now also U31.J19 (IO_L10N_T1_AD11N_35)
- net DATA3-11_0: now also U31.P20 (IO_L14N_T2_SRCC_34)
- net DATA3-13_0: now also U31.R18 (IO_L20N_T3_34)
- net DATA3-14_0: now also U31.R19 (IO_0_34)
- net DATA3-15_0: now also U31.P19 (IO_L13N_T2_MRCC_34)
- net DATA3-16_0: now also U31.T20 (IO_L15P_T2_DQS_34)
- net DATA3-17_0: now also U31.U20 (IO_L15N_T2_DQS_34)
- net DATA3-18_0: now also U31.T19 (IO_25_34)
- net DATA3-19_0: now also U31.V20 (IO_L16P_T2_34)
- net DATA3-20_0: now also U31.U19 (IO_L12N_T1_MRCC_34)
- net DATA3-5_0: now also U31.M19 (IO_L7P_T1_AD2P_35)
- net DATA3-6_0: now also U31.N20 (IO_L14P_T2_SRCC_34)
- net DATA3-7_0: now also U31.P18 (IO_L23N_T3_34)
- net DATA3-8_0: now also U31.M17 (IO_L8P_T1_AD10P_35)
- net DATA3-9_0: now also U31.N17 (IO_L23P_T3_34)
- net DDR-A0_0: now also U66.N3 (A0)
- net DDR-A10_0: now also U66.L7 (A10/AP)
- net DDR-A11_0: now also U66.R7 (A11)
- net DDR-A12_0: now also U66.N7 (A12/~BC~)
- net DDR-A13_0: now also U66.T3 (A13)
- net DDR-A14_0: now also U66.T7 (NC)
- net DDR-A1_0: now also U66.P7 (A1)
- net DDR-A2_0: now also U66.P3 (A2)
- net DDR-A3_0: now also U66.N2 (A3)
- net DDR-A4_0: now also U66.P8 (A4)
- net DDR-A5_0: now also U66.P2 (A5)
- net DDR-A6_0: now also U66.R8 (A6)
- net DDR-A7_0: now also U66.R2 (A7)
- net DDR-A8_0: now also U66.T8 (A8)
- net DDR-A9_0: now also U66.R3 (A9)
- net DDR-BA0_0: now also U66.M2 (BA0)
- net DDR-BA1_0: now also U66.N8 (BA1)
- net DDR-BA2_0: now also U66.M3 (BA2)
- net DDR-CAS_0: now also U66.K3 (~CAS~)
- net DDR-CK#_0: now also U31.M2 (PS_DDR_CKN_502), U66.K7 (~CK~)
- net DDR-CKE_0: now also U66.K9 (CKE)
- net DDR-CK_0: now also U31.L2 (PS_DDR_CKP_502), U66.J7 (CK)
- net DDR-CS_0: now also U66.L2 (~CS~)
- net DDR-DQ0_0: now also U31.C3 (PS_DDR_DQ0_502), U66.E3 (DQ0)
- net DDR-DQ10_0: now also U31.G3 (PS_DDR_DQ10_502), U66.C8 (DQ10)
- net DDR-DQ11_0: now also U31.H3 (PS_DDR_DQ11_502), U66.C2 (DQ11)
- net DDR-DQ12_0: now also U31.J3 (PS_DDR_DQ12_502), U66.A7 (DQ12)
- net DDR-DQ13_0: now also U31.H2 (PS_DDR_DQ13_502), U66.A2 (DQ13)
- net DDR-DQ14_0: now also U31.H1 (PS_DDR_DQ14_502), U66.B8 (DQ14)
- net DDR-DQ15_0: now also U31.J1 (PS_DDR_DQ15_502), U66.A3 (DQ15)
- net DDR-DQ1_0: now also U31.B3 (PS_DDR_DQ1_502), U66.F7 (DQ1)
- net DDR-DQ2_0: now also U31.A2 (PS_DDR_DQ2_502), U66.F2 (DQ2)
- net DDR-DQ3_0: now also U31.A4 (PS_DDR_DQ3_502), U66.F8 (DQ3)
- net DDR-DQ4_0: now also U31.D3 (PS_DDR_DQ4_502), U66.H3 (DQ4)
- net DDR-DQ5_0: now also U31.D1 (PS_DDR_DQ5_502), U66.H8 (DQ5)
- net DDR-DQ6_0: now also U31.C1 (PS_DDR_DQ6_502), U66.G2 (DQ6)
- net DDR-DQ7_0: now also U31.E1 (PS_DDR_DQ7_502), U66.H7 (DQ7)
- net DDR-DQ8_0: now also U31.E2 (PS_DDR_DQ8_502), U66.D7 (DQ8)
- net DDR-DQ9_0: now also U31.E3 (PS_DDR_DQ9_502), U66.C3 (DQ9)
- net DDR-LDM_0: now also U31.A1 (PS_DDR_DM0_502), U66.E7 (LDM)
- net DDR-LDQS#_0: now also U31.B2 (PS_DDR_DQS_N0_502), U66.G3 (~LDQS~)
- net DDR-LDQS_0: now also U31.C2 (PS_DDR_DQS_P0_502), U66.F3 (LDQS)
- net DDR-ODT_0: now also U66.K1 (ODT)
- net DDR-RAS_0: now also U66.J3 (~RAS~)
- net DDR-RESET_0: now also U31.B4 (PS_DDR_DRST_B_502), U66.T2 (~RESET~)
- net DDR-UDM_0: now also U31.F1 (PS_DDR_DM1_502), U66.D3 (UDM)
- net DDR-UDQS#_0: now also U31.F2 (PS_DDR_DQS_N1_502), U66.B7 (~UDQS~)
- net DDR-UDQS_0: now also U31.G2 (PS_DDR_DQS_P1_502), U66.C7 (UDQS)
- net DDR-WE_0: now also U66.L3 (~WE~)
- net GND: now also U12.13 (VSS_1), U12.36 (VSS_2), U22.1 (GND), U24.11 (DGND), U24.17 (DGND), U24.29 (AGND1V), U24.35 (AGND33), U24.40 (NC), U24.43 (TXER/FXSD), U24.45 (DGND), U26.1 (GND), U27.1 (GND), U28.1 (GND), U30.1 (GND), U31.A18 (GND), U31.A8 (GND), U31.B1 (GND), U31.B11 (GND), U31.C14 (GND), U31.C4 (GND), U31.C9 (GND), U31.D17 (GND), U31.E10 (GND), U31.E20 (GND), U31.F10 (RSVDGND), U31.F3 (GND), U31.F7 (GND), U31.G10 (GND), U31.G12 (GND), U31.G16 (GND), U31.H11 (GND), U31.H13 (GND), U31.H19 (GND), U31.H7 (GND), U31.H9 (GND), U31.J12 (GND), U31.J2 (GND), U31.J8 (GND), U31.K11 (GND), U31.K13 (GND), U31.K15 (GND), U31.K5 (GND), U31.K7 (GND), U31.K9 (VP_0), U31.L10 (VN_0), U31.L12 (GND), U31.L18 (GND), U31.L8 (GND), U31.M1 (GND), U31.M10 (DXN_0), U31.M11 (GND), U31.M13 (GND), U31.M7 (GND), U31.M9 (DXP_0), U31.N10 (GND), U31.N12 (GND), U31.N14 (GND), U31.N4 (GND), U31.N8 (GND), U31.P11 (GND), U31.P13 (GND), U31.P17 (GND), U31.P7 (GND), U31.P9 (GND), U31.R12 (GND), U31.R20 (GND), U31.R8 (GND), U31.T13 (GND), U31.T3 (GND), U31.T7 (GND), U31.U16 (GND), U31.U6 (GND), U31.V19 (GND), U31.V9 (GND), U31.W12 (GND), U31.W2 (GND), U31.Y15 (GND), U31.Y5 (GND), U65.3 (GND), U66.A9 (VSS), U66.B1 (VSSQ), U66.B3 (VSS), U66.B9 (VSSQ), U66.D1 (VSSQ), U66.D8 (VSSQ), U66.E1 (VSS), U66.E2 (VSSQ), U66.E8 (VSSQ), U66.F9 (VSSQ), U66.G1 (VSSQ), U66.G8 (VSS), U66.G9 (VSSQ), U66.J2 (VSS), U66.J8 (VSS), U66.M1 (VSS), U66.M9 (VSS), U66.P1 (VSS), U66.P9 (VSS), U66.T1 (VSS), U66.T9 (VSS), U67.3, U68.3, U7.10 (MNT1), U7.11 (MNT2), U7.12 (MNT3), U7.13 (MNT4), U7.6 (VSS), U72.11 (EP_3), U72.12 (EP_4), U72.13 (EP_1), U72.14 (EP_2), U72.15 (EP_5), U72.4 (PGND), U72.8 (GND), X3.4 (GND), X5.4 (GND), X8.2 (GND), Y2.5, Y2.6
- net GND3: now also U69.3, U70.3
- net GNDADC_0: now also U31.J10 (GNDADC_0), U31.K10 (VREFN_0)
- net IN: now also U22.3 (IN), U26.3 (IN), U27.3 (IN), U28.3 (IN)
- net LED.0_0: now also U24.9 (LED0/PHY_AD0), U25.11
- net LED3_0: now also U24.13 (LED3/PHY_AD3), U25.9
- net MDC_0: now also U24.25 (MDC), U31.W15 (IO_L10N_T1_34)
- net NetC2300_2: now also U66.H1 (VREFDQ), U66.M8 (VREFCA)
- net NetC327_1: now also U31.J9 (VCCADC_0)
- net NetC69_1: now also X3.1 (X1), Y2.1, Y2.8
- net NetLED6_1: now also LED6.1 (A1)
- net NetLED6_2: now also LED6.2 (A2)
- net NetR117_2: now also X3.3 (VBAT)
- net NetR1345_1: now also U67.2
- net NetR1346_1: now also U69.4
- net NetR1360_1: now also U12.19 (#WP)
- net NetR1362_1: now also U68.2
- net NetR1363_1: now also U70.4
- net NetR1372_1: now also X5.3 (OUT)
- net NetR1372_2: now also U31.N18 (IO_L13P_T2_MRCC_34)
- net NetR1384_2: now also T6.10 (RXCT)
- net NetR1385_2: now also U24.22 (RXDV/CRS_DV/FX_HEN)
- net NetR1393_1: now also U24.28 (ISET)
- net NetR1400_2: now also T6.15 (TXCT)
- net NetR1413_2: now also U26.5 (EN)
- net NetR1493_1: now also U31.F11 (VCCBATT_0)
- net NetR1500_1: now also U31.R11 (DONE_0)
- net NetR1502_1: now also U31.L6 (PROGRAM_B_0)
- net NetR1503_1: now also U31.R10 (INIT_B_0)
- net NetR1949_2: now also U65.4 (PFI)
- net NetR2336_1: now also U65.1 (~MR)
- net NetR2340_2: now also X8.3 (OUT)
- net NetR2389_1: now also X8.1 (EN)
- net NetR2430_1: now also U31.B10 (PS_SRST_B_501)
- net NetR2433_1: now also U31.E11 (PS_MIO_VREF_501)
- net NetR2455_1: now also U66.L8 (ZQ)
- net NetR2461_2: now also U31.U15 (IO_L11N_T1_SRCC_34)
- net NetR2462_2: now also U31.W19 (IO_L22N_T3_34)
- net NetR2463_2: now also U31.W18 (IO_L22P_T3_34)
- net NetR2464_2: now also U31.Y18 (IO_L17P_T2_34)
- net NetR2466_2: now also U31.Y19 (IO_L17N_T2_34)
- net NetR2468_1: now also U23.1
- net NetR2540_1: now also U31.U13 (IO_L3P_T0_DQS_PUDC_B_34)
- net NetR2545_2: now also U67.1
- net NetR2547_2: now also U68.1
- net NetR2605_1: now also U28.5 (EN)
- net NetR2615_1: now also U72.1 (REFIN)
- net NetR2618_2: now also U72.5 (VOSNS)
- net NetT6_1: now also T6.1 (TD+), U24.34 (MDI_TP)
- net NetT6_3: now also T6.3 (TD-), U24.33 (MDI_TN)
- net NetT6_6: now also T6.6 (RD+), U24.31 (MDI_RP)
- net NetT6_8: now also T6.8 (RD-), U24.30 (MDI_RN)
- net NetU12_25: now also U12.25 (N.C_15)
- net NetU12_34: now also U12.34 (N.C_20)
- net NetU12_38: now also U12.38 (DNU_2)
- net NetU12_39: now also U12.39 (N.C_22)
- net NetU12_48: now also U12.48 (N.C_27)
- net NetU22_2: now also U22.2 (SW)
- net NetU22_4: now also U22.4 (FB)
- net NetU22_5: now also U22.5 (EN)
- net NetU22_6: now also U22.6 (S)
- net NetU24_10: now also U24.10 (LED1/PHY_AD1)
- net NetU24_12: now also U24.12 (LED2/PHY_AD2)
- net NetU24_15: now also U24.15 (NC)
- net NetU24_16: now also U24.16 (RXCLK/50M_CLKO)
- net NetU24_18: now also U24.18 (RXD3)
- net NetU24_19: now also U24.19 (RXD2)
- net NetU24_20: now also U24.20 (RXD1)
- net NetU24_21: now also U24.21 (RXD0)
- net NetU24_23: now also U24.23 (CRS/LEDMOD)
- net NetU24_24: now also U24.24 (RXER)
- net NetU24_46: now also U24.46 (X1)
- net NetU24_47: now also U24.47 (X2)
- net NetU25_1: now also T6.16 (TX+), U25.1
- net NetU25_10: now also U25.10
- net NetU25_12: now also U25.12
- net NetU25_2: now also T6.14 (TX-), U25.2
- net NetU25_3: now also T6.11 (RX+), U25.3
- net NetU25_4: now also U25.4, U25.5
- net NetU25_6: now also T6.9 (RX-), U25.6
- net NetU25_7: now also U25.7, U25.8
- net NetU26_2: now also U26.2 (SW)
- net NetU26_4: now also U26.4 (FB)
- net NetU26_6: now also U26.6 (S)
- net NetU27_2: now also U27.2 (SW)
- net NetU27_4: now also U27.4 (FB)
- net NetU27_5: now also U27.5 (EN)
- net NetU27_6: now also U27.6 (S)
- net NetU28_2: now also U28.2 (SW)
- net NetU28_4: now also U28.4 (FB)
- net NetU28_6: now also U28.6 (S)
- net NetU30_2: now also U30.2 (~RESET)
- net NetU30_3: now also U30.3 (VDD)
- net NetU31_A16: now also U31.A16 (PS_MIO24_501)
- net NetU31_A19: now also U31.A19 (PS_MIO16_501)
- net NetU31_B12: now also U31.B12 (PS_MIO48_501)
- net NetU31_B13: now also U31.B13 (PS_MIO50_501)
- net NetU31_B14: now also U31.B14 (PS_MIO47_501)
- net NetU31_B18: now also U31.B18 (PS_MIO18_501)
- net NetU31_C12: now also U31.C12 (PS_MIO49_501)
- net NetU31_C13: now also U31.C13 (PS_MIO29_501)
- net NetU31_C15: now also U31.C15 (PS_MIO30_501)
- net NetU31_C16: now also U31.C16 (PS_MIO28_501)
- net NetU31_C18: now also U31.C18 (PS_MIO39_501)
- net NetU31_D16: now also U31.D16 (PS_MIO46_501)
- net NetU31_E13: now also U31.E13 (PS_MIO38_501)
- net NetU31_E16: now also U31.E16 (PS_MIO31_501)
- net NetU31_F12: now also U31.F12 (PS_MIO35_501)
- net NetU31_F15: now also U31.F15 (PS_MIO25_501)
- net NetU31_G5: now also U31.G5 (PS_DDR_VRN_502)
- net NetU31_G8: now also U31.G8 (VCCPLL)
- net NetU31_H5: now also U31.H5 (PS_DDR_VRP_502)
- net NetU31_H6: now also U31.H6 (PS_DDR_VREF0_502)
- net NetU31_N6: now also U31.N6 (RSVDVCC3)
- net NetU31_P6: now also U31.P6 (PS_DDR_VREF1_502)
- net NetU31_R6: now also U31.R6 (RSVDVCC2)
- net NetU31_T6: now also U31.T6 (RSVDVCC1)
- net NetU31_V18: now also U31.V18 (IO_L21N_T3_DQS_34)
- net NetU65_7: now also U65.7 (~RESET)
- net NetU69_1: now also U69.1
- net NetU70_1: now also U70.1
- net NetU72_6: now also U72.6 (REFOUT)
- net NetU72_7: now also U72.7 (EN)
- net NetU72_9: now also U72.9 (PGOOD)
- net NetU7_9: now also U7.9 (DETECT)
- net NetX3_5: now also X3.5 (SDA)
- net NetX3_6: now also X3.6 (SCL)
- net NetX3_7: now also X3.7 (SQW/OUT)
- net NetX5_1: now also X5.1 (EN)
- net NetX5_2: now also X5.2 (Vdd)
- net NetX8_4: now also X8.4 (Vdd)
- net NetY2_7: now also X3.2 (X2), Y2.2, Y2.7
- net PS-DDR-A0_0: now also U31.N2 (PS_DDR_A0_502)
- net PS-DDR-A10_0: now also U31.F5 (PS_DDR_A10_502)
- net PS-DDR-A11_0: now also U31.G4 (PS_DDR_A11_502)
- net PS-DDR-A12_0: now also U31.E4 (PS_DDR_A12_502)
- net PS-DDR-A13_0: now also U31.D4 (PS_DDR_A13_502)
- net PS-DDR-A14_0: now also U31.F4 (PS_DDR_A14_502)
- net PS-DDR-A1_0: now also U31.K2 (PS_DDR_A1_502)
- net PS-DDR-A2_0: now also U31.M3 (PS_DDR_A2_502)
- net PS-DDR-A3_0: now also U31.K3 (PS_DDR_A3_502)
- net PS-DDR-A4_0: now also U31.M4 (PS_DDR_A4_502)
- net PS-DDR-A5_0: now also U31.L1 (PS_DDR_A5_502)
- net PS-DDR-A6_0: now also U31.L4 (PS_DDR_A6_502)
- net PS-DDR-A7_0: now also U31.K4 (PS_DDR_A7_502)
- net PS-DDR-A8_0: now also U31.K1 (PS_DDR_A8_502)
- net PS-DDR-A9_0: now also U31.J4 (PS_DDR_A9_502)
- net PS-DDR-BA0_0: now also U31.L5 (PS_DDR_BA0_502)
- net PS-DDR-BA1_0: now also U31.R4 (PS_DDR_BA1_502)
- net PS-DDR-BA2_0: now also U31.J5 (PS_DDR_BA2_502)
- net PS-DDR-CAS_0: now also U31.P5 (PS_DDR_CAS_B_502)
- net PS-DDR-CKE_0: now also U31.N3 (PS_DDR_CKE_502)
- net PS-DDR-CS_0: now also U31.N1 (PS_DDR_CS_B_502)
- net PS-DDR-ODT_0: now also U31.N5 (PS_DDR_ODT_502)
- net PS-DDR-RAS_0: now also U31.P4 (PS_DDR_RAS_B_502)
- net PS-DDR-WE_0: now also U31.M5 (PS_DDR_WE_B_502)
- net REGOUT: now also U24.8 (REGOUT)
- net REGOUT.0: now also T6.2 (TCT), T6.7 (RCT), U24.32 (NC)
- net RESET.0_0: now also U31.C7 (PS_POR_B_500)
- net RESET.1_0: now also U24.42 (~RESET_N)
- net REST.ON_0: now also U24.26 (MDIO), U31.Y14 (IO_L8N_T1_34)
- net RXCLK_0: now also U31.U14 (IO_L11P_T1_SRCC_34)
- net RXD0_0: now also U31.Y16 (IO_L7P_T1_34)
- net RXD1_0: now also U31.V16 (IO_L18P_T2_34)
- net RXD2_0: now also U31.V17 (IO_L21P_T3_DQS_34)
- net RXD3_0: now also U31.Y17 (IO_L7N_T1_34)
- net RXDV_0: now also U31.W16 (IO_L18N_T2_34)
- net RY/#BY_0: now also U12.7 (RY/#BY), U31.C5 (PS_MIO14_500)
- net TXCLK_0: now also U24.7 (TXCLK/50M_CLKI)
- net TXD0_0: now also U24.6 (TXD0)
- net TXD1_0: now also U24.5 (TXD1)
- net TXD2_0: now also U24.4 (TXD2)
- net TXD3_0: now also U24.3 (TXD3)
- net TXEN_0: now also U24.2 (TXEN)
- net U12-IO0_0: now also U12.29 (IO0), U31.A6 (PS_MIO5_500)
- net U12-IO1_0: now also U12.30 (IO1), U31.A5 (PS_MIO6_500)
- net U12-IO2_0: now also U12.31 (IO2), U31.B7 (PS_MIO4_500)
- net U12-IO3_0: now also U12.32 (IO3), U31.E8 (PS_MIO13_500)
- net U12-IO4_0: now also U12.41 (IO4), U31.B5 (PS_MIO9_500)
- net U12-IO5_0: now also U12.42 (IO5), U31.E9 (PS_MIO10_500)
- net U12-IO6_0: now also U12.43 (IO6), U31.C6 (PS_MIO11_500)
- net U12-IO7_0: now also U12.44 (IO7), U31.D9 (PS_MIO12_500)
- net U3.A.12_0: now also U31.A12 (PS_MIO34_501)
- net U3.A.9_0: now also U31.A9 (PS_MIO43_501), U7.8 (DAT1)
- net U3.A14_0: now also U31.A14 (PS_MIO32_501)
- net U3.A17_0: now also U31.A17 (PS_MIO20_501)
- net U3.B.15_0: now also U31.B15 (PS_MIO45_501), U7.2 (DAT3/CD)
- net U3.C.17_0: now also U31.C17 (PS_MIO41_501), U7.3 (CMD)
- net U3.D.14_0: now also U31.D14 (PS_MIO40_501), U7.5 (CLK)
- net U3.E.12_0: now also U31.E12 (PS_MIO42_501), U7.7 (DAT0)
- net U3.F13_0: now also U31.F13 (PS_MIO44_501), U7.1 (DAT2)
- net U3.U12_0: now also U31.U12 (IO_L2N_T0_34), U69.2
- net U3.V12_0: now also U31.V12 (IO_L4P_T0_34), U70.2
- net U3.V13_0: now also U31.V13 (IO_L3N_T0_DQS_34), U67.4
- net U3.V15_0: now also U31.V15 (IO_L10P_T1_34), U68.4
- net U3.W13_0: now also LED6.4 (K1), U31.W13 (IO_L4N_T0_34)
- net U3.W14_0: now also LED6.3 (K2), U31.W14 (IO_L8P_T1_34)
- net U31-A15_0: now also U31.A15 (PS_MIO26_501)
- net U31-D13_0: now also U31.D13 (PS_MIO27_501)
- net U31-L14_0: now also U31.L14 (IO_L22P_T3_AD7P_35)
- net U31-N16_0: now also U31.N16 (IO_L21N_T3_DQS_AD14N_35)
- net U31-TCK_0: now also U31.F9 (TCK_0)
- net U31-TDI_0: now also U31.G6 (TDI_0)
- net U31-TDO_0: now also U31.F6 (TDO_0)
- net U31-TMS_0: now also U31.J6 (TMS_0)
- net U31.W20_0: now also U31.W20 (IO_L16N_T2_34)
- net VCC: now also U12.12 (VCC_1), U12.37 (VCC_2), U23.3, U24.14 (VDDIO), U24.36 (AVDD33), U24.41 (NC), U24.44 (NC), U24.48 (INTR), U31.A13 (VCCO_MIO1_501), U31.B16 (VCCO_MIO1_501), U31.B6 (VCCO_MIO0_500), U31.D12 (VCCO_MIO1_501), U31.D7 (VCCO_MIO0_500), U31.E15 (VCCO_MIO1_501), U31.M6 (CFGBVS_0), U31.T8 (VCCO_13), U31.U11 (VCCO_13), U31.W7 (VCCO_13), U31.Y10 (VCCO_13), U65.2 (VCC), U7.4 (VDD), U72.10 (VIN)
- net VCC-DDR: now also U31.A3 (VCCO_DDR_502), U31.D2 (VCCO_DDR_502), U31.E5 (VCCO_DDR_502), U31.G1 (VCCO_DDR_502), U31.H4 (VCCO_DDR_502), U31.L3 (VCCO_DDR_502), U31.P2 (VCCO_DDR_502), U31.R5 (VCCO_DDR_502), U31.U1 (VCCO_DDR_502), U31.V4 (VCCO_DDR_502), U66.A1 (VDDQ), U66.A8 (VDDQ), U66.B2 (VDD), U66.C1 (VDDQ), U66.C9 (VDDQ), U66.D2 (VDDQ), U66.D9 (VDD), U66.E9 (VDDQ), U66.F1 (VDDQ), U66.G7 (VDD), U66.H2 (VDDQ), U66.H9 (VDDQ), U66.K2 (VDD), U66.K8 (VDD), U66.N1 (VDD), U66.N9 (VDD), U66.R1 (VDD), U66.R9 (VDD), U72.2 (VLDOIN)
- net VCC1: now also U72.3 (VO)
- net VCC6: now also X3.8 (VCC)
- net VCCA: now also U31.F8 (VCCPAUX), U31.G9 (VCCPAUX), U31.H8 (VCCPAUX), U31.J11 (VCCAUX), U31.K8 (VCCPAUX), U31.L11 (VCCAUX), U31.M8 (VCCPAUX), U31.N11 (VCCAUX), U31.N9 (VCCAUX), U31.P10 (VCCAUX), U31.R9 (VCCAUX)
- net VCCB: now also U31.K6 (VCCO_0)
- net VCCE: now also U31.N19 (VCCO_34), U31.R15 (VCCO_34), U31.T18 (VCCO_34), U31.V14 (VCCO_34), U31.W17 (VCCO_34), U31.Y20 (VCCO_34)
- net VCCO: now also U31.C19 (VCCO_35), U31.F18 (VCCO_35), U31.H14 (VCCO_35), U31.J17 (VCCO_35), U31.K20 (VCCO_35), U31.M16 (VCCO_35)
- net VCCP: now also U31.G11 (VCCBRAM), U31.G13 (VCCINT), U31.G7 (VCCPINT), U31.H10 (VCCBRAM), U31.H12 (VCCINT), U31.J13 (VCCINT), U31.J7 (VCCPINT), U31.K12 (VCCINT), U31.L13 (VCCINT), U31.L7 (VCCPINT), U31.M12 (VCCINT), U31.N13 (VCCINT), U31.N7 (VCCPINT), U31.P12 (VCCINT), U31.P8 (VCCPINT), U31.R13 (VCCINT), U31.R7 (VCCPINT)
- net VP1_0: now also U23.2, U23.4, U31.L9 (VREFP_0)
- net XOUT.0_0: now also U31.U18 (IO_L12P_T1_MRCC_34)

Commit message: Implemented component grouping by schematic section.
It's quick & dirty, but it does the job.
Other:
- note added: "DDR"
- note added: "DDR Termination"
- note added: "Data Conns"
- note added: "Ethernet PHY"
- note added: "Flash"
- note added: "Opto-Isolators"
- note added: "Power"
- note added: "RTC"
- note added: "Reset Supervisor"
- note added: "SD and Ancillary"
- note added: "Switches"
- note added: "Zynq"
- note added: "Zynq IO"
- note added: "Zynq Oscs"
- note added: "Zynq Power"
